File: modules/mco/mco.kicad_sch (KiCad schematic)
At the start: 25 parts, among them U1 ATtiny1616-M, U3 MCP6002-xSN

Commit message: mco: Add MIDI THRU support
Parts:
- removed R5, R7: 1k, Resistor_SMD:R_0402_1005Metric, symbol Device:R
Connections:
- net DETUNED_OUT is gone; now on net VELOCITY: OUTPUT1.5 (Pin_5)
- net SQUARE_OUT is gone; now on net GATE: OUTPUT1.4 (Pin_4)
- net GATE: no longer OUTPUT1.2 (Pin_2)
- net MIDI: now also OUTPUT1.1 (Pin_1)
- net MIX_OUT: now also OUTPUT1.2 (Pin_2), OUTPUT1.3 (Pin_3); no longer OUTPUT1.1 (Pin_1)
- net VELOCITY: no longer OUTPUT1.3 (Pin_3)
