File: modules/drive/drive.kicad_pcb (KiCad board)
At the start: 2 copper layers, 30.5 x 68.6 mm, 23 parts, among them U1 MCP6002-xSN

Commit message: drive_1.0.0
Other:
- board text added: "DRIVE 1.0.0"
- board text removed: "DRIVE 0.2.0"
Changed lines of the file:
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@@
 		)
 	)
-	(gr_text "DRIVE\n0.2.0"
+	(gr_text "DRIVE\n1.0.0"
 		(at 76.327 107.95 0)
 		(layer "F.SilkS")
