File: modules/svf/svf.kicad_pcb (KiCad board)
At the start: 2 copper layers, 30.5 x 68.6 mm, 34 parts, among them U1 VTL5C, U2 VTL5C, U3 MCP6002-xSN, U4 MCP6002-xSN, U5 MCP6002-xSN

Commit message: svf_1.0.0
Other:
- board text added: "SVF 1.0.0"
- board text removed: "SVF 0.2.0"
Changed lines of the file:
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@@
 		(tags "resistor")
 		(property "Reference" "R9"
-			(at -0.002 -1.27 360)
+			(at -0.002 -1.27 0)
 			(layer "F.SilkS")
 			(effects
@@
 		)
 		(property "Value" "1k"
-			(at 0 1.17 360)
+			(at 0 1.17 0)
 			(layer "F.Fab")
 			(effects
@@
 		)
 		(fp_text user "${REFERENCE}"
-			(at 0 0 360)
+			(at 0 0 0)
 			(layer "F.Fab")
 			(effects
@@
 		)
 		(property "Value" "1k"
-			(at 0 1.17 360)
+			(at 0 1.17 0)
 			(layer "F.Fab")
 			(effects
@@
 		)
 		(fp_text user "${REFERENCE}"
-			(at 0 0 360)
+			(at 0 0 0)
 			(layer "F.Fab")
 			(effects
@@
 		)
 	)
-	(gr_text "SVF\n0.2.0"
+	(gr_text "SVF\n1.0.0"
 		(at 76.327 107.95 0)
 		(layer "F.SilkS")
