File: opt/UPDIProgrammer/UPDIProgrammer.kicad_pcb (KiCad board)
At the start: 2 copper layers, 34.3 x 17.1 mm, 21 parts, among them J2 USB_C_Receptacle_USB2.0_14P, U1 CH340N, U2 ATtiny1616-M

Commit message: Update the UPDI Programmer.
Parts:
- removed VSUPPLY1: Conn_01x05_Pin, Connector_PinHeader_2.54mm:PinHeader_1x05_P2.54mm_Vertical
- added NC1: Conn_01x05_Pin, Connector_PinHeader_2.54mm:PinHeader_1x05_P2.54mm_Vertical, B.Cu at (223.5, 45.7)
- added R9: 330, Resistor_SMD:R_0402_1005Metric, F.Cu at (214.9, 43.2)
Connections:
- GND1 pad 1: GND -> Net-(GND1-Pin_1)
- GND1 pad 2: GND -> Net-(GND1-Pin_1)
- GND1 pad 3: GND -> Net-(GND1-Pin_1)
- GND1 pad 4: GND -> Net-(GND1-Pin_1)
- GND1 pad 5: GND -> Net-(GND1-Pin_1)
Routing:
- net +3.3V: track 25.1 -> 0.00 mm
- net Net-(GND1-Pin_1): track 0.00 -> 22.3 mm, vias 0 -> 1
- net GND: track 169.3 -> 153.7 mm, vias 10 -> 11
- net Net-(NC1-Pin_1): track 0.00 -> 10.2 mm
- net 5V: track 32.1 -> 32.8 mm
Other:
- board text added: "UPDI"
- board text added: "UPDI 0.3.0"
- board text removed: "UDPI"
- board text removed: "UDPI 0.2.0"
