File: modules/low/low.kicad_sch (KiCad schematic)
At the start: 31 parts, among them U1 VTL5C, U2 MCP6002-xSN, U3 VTL5C, U4 VTL5C, U5 MCP6002-xSN

Commit message: low: Add the new design and renamed it to low
Parts:
- removed R10: 10k, Resistor_SMD:R_0402_1005Metric, symbol Device:R
- removed R8: 560, Resistor_SMD:R_0402_1005Metric, symbol Device:R
- removed R9: 1M, Resistor_SMD:R_0402_1005Metric, symbol Device:R
- removed RV1: 1M, BreadModular_Pots:Potentiometer_RV09, symbol Device:R_Potentiometer
- removed U4: VTL5C, BreadModular_MISC:VTL5C, symbol Isolator:VTL5C
- removed V3: 3.3, symbol Simulation_SPICE:VDC
- added SW1: SPST_TS-1187A-B-A-B, BreadModular_MISC:SPST_TS-1187A-B-A-B, symbol Switch:SW_SPST
- R3: value 560 -> 1M
- R4: value 200k -> 1M
- R6, R7: value 200k -> 330
- RV1: renamed from RV2; value 1M -> 50k; Comment CUT_OFF_CURVE -> CUT_OFF
Connections:
- net GND: now also R4.1, R6.2; no longer INPUT1.5 (Pin_5), RV1.2, U1.1 (-), U3.1 (-)
- net VAC_NEG: now reaches U5.2 (-)
- net VAC_NEG: now also RV1.2, U1.1 (-), U3.1 (-), SW1.1 (A); no longer U5.1
- net at U5.6 (-), U5.7: now also R3.2; no longer R7.1
- net at R4.2: now also R3.1, U5.3 (+); no longer R3.2
- net at R6.1, R7.2: now also RV1.3
- net VAC_POS: now reaches U1.2 (+), U3.2 (+)
- net VAC_POS: now also U5.1; no longer R3.1
- net at R12.2: now also INPUT1.3 (Pin_3); no longer INPUT1.4 (Pin_4)
- removed net CUT_OFF_CV: INPUT1.3 (Pin_3), U5.3 (+)
- net GATE_CV renamed CV
- new net: R7.1, SW1.2 (B)
Other:
- note added: "## 2. CV Input We can feed either CV or a GATE input here. If it's a GATE this will act as a low pass gate."
- note added: "## 3. Cutt Off This act as a cutoff point of the filter. pos=0 => lower end of the freq. spectrum pos=1 => higher end of the freq. spectrum We can feed +V_SUPPLY to the CV and then, we can turn this into a low pass filter."
- note added: "## 4. Blast This will set CUT_OFF pos=1.0 momentarly. It's very cool, performance feature."
- note removed: "## 2. Gate CV This is the CV that drives filter resistors. Since those are Vactrols, 0-VMax CV both does filter cut off modulation and act as a VCA. Here RV1, put a cap to where vactrol can drive. So, technically it's the cutt-off point controlled by a pot. pos=0.0 => low frequency pos=1.0 => high frequency"
- note removed: "## 3. Cut Off CV This is another set of CV modulation, but it's changing the Cut Off position. (Just like rotating the RV1) Now RV2 act as changing the curve of CV. * pos=0.0 => Exponential Curve * pos=1.0 => Linear Curve"
- moved on the sheet: C2, C3, R11, R5, RV1, U1, U2A, U2B, U3, U5A, U5B, V1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

Commit message: low: Change the push button
Parts:
- SW1: value SPST_TS-1187A-B-A-B -> K2-1808SN-A4SW-01; footprint BreadModular_MISC:SPST_TS-1187A-B-A-B -> BreadModular_MISC:K2-1808SN-A4SW-01
Changed lines of the file:
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@@
 			)
 		)
-		(property "Value" "SPST_TS-1187A-B-A-B"
+		(property "Value" "K2-1808SN-A4SW-01"
 			(at 111.76 227.33 0)
 			(effects
@@
 			)
 		)
-		(property "Footprint" "BreadModular_MISC:SPST_TS-1187A-B-A-B"
+		(property "Footprint" "BreadModular_MISC:K2-1808SN-A4SW-01"
 			(at 111.76 231.14 0)
 			(effects
