File: opt/Breakouts/RP2350A/RP2350_60QFN_minimal.kicad_sch (KiCad schematic)
At the start: 42 parts, among them J1 Conn_01x16_Socket, J2 Conn_01x16_Socket, J5 USB_C_Receptacle_USB2.0_14P, SW1 SW_SPST, SW3 K2-1808SN-A4SW-01, U1 RP2350_60QFN, U2 W25Q128JVS, Y1 ABM8-272-T3

Commit message: Finished building the RP2350 module
Parts:
- removed H1, H2, H3, H4: MountingHole, MountingHole:MountingHole_2.7mm_M2.5, symbol Mechanical:MountingHole
- removed J1, J2: Conn_01x16_Socket, Connector_PinSocket_2.54mm:PinSocket_1x16_P2.54mm_Vertical, symbol Connector:Conn_01x16_Socket
- added D1: LED, LED_SMD:LED_0603_1608Metric, symbol Device:LED
- added J1, J2: Conn_01x08_Socket, Connector_PinSocket_2.54mm:PinSocket_1x08_P2.54mm_Vertical, symbol Connector:Conn_01x08_Socket
- added R9: 1k, Resistor_SMD:R_0402_1005Metric, symbol Device:R
- added SW2: K2-1808SN-A4SW-01, BreadModular_MISC:K2-1808SN-A4SW-01, symbol Switch:SW_SPST
- SW1: Comment (none) -> RESET
- SW3: Comment (none) -> BOOT
- renumbered 5V1 to V_SUPPLY1
Connections:
- net GND: now also R9.1, SW2.2 (B)
- net GPIO0: now also J1.1 (Pin_1)
- net GPIO1: now also J1.2 (Pin_2)
- net GPIO12: now also SW2.1 (A)
- net GPIO13: now also D1.2 (A)
- net GPIO2: now also J1.3 (Pin_3)
- net GPIO25: now also J2.5 (Pin_5)
- net GPIO26_ADC0: now also J2.4 (Pin_4)
- net GPIO27_ADC1: now also J2.3 (Pin_3)
- net GPIO28_ADC2: now also J2.2 (Pin_2)
- net GPIO29_ADC3: now also J2.1 (Pin_1)
- net GPIO3: now also J1.4 (Pin_4)
- net GPIO4: now also J1.5 (Pin_5)
- net GPIO5: now also J1.6 (Pin_6)
- net GPIO6: now also J1.7 (Pin_7)
- net GPIO7: now also J1.8 (Pin_8)
- net RUN: now also J2.6 (Pin_6)
- net SWCLK: now also J2.8 (Pin_8)
- net SWD: now also J2.7 (Pin_7)
- net GPIO10: no longer names the net of U1.14 (GPIO10)
- net GPIO11: no longer names the net of U1.15 (GPIO11)
- net GPIO14: no longer names the net of U1.18 (GPIO14)
- net GPIO15: no longer names the net of U1.19 (GPIO15)
- net GPIO17: no longer names the net of U1.28 (GPIO17)
- net GPIO18: no longer names the net of U1.29 (GPIO18)
- net GPIO19: no longer names the net of U1.31 (GPIO19)
- net GPIO20: no longer names the net of U1.32 (GPIO20)
- net GPIO21: no longer names the net of U1.33 (GPIO21)
- net GPIO22: no longer names the net of U1.34 (GPIO22)
- net GPIO23: no longer names the net of U1.35 (GPIO23)
- net GPIO24: no longer names the net of U1.36 (GPIO24)
- net GPIO8: no longer names the net of U1.12 (GPIO8)
- net GPIO9: no longer names the net of U1.13 (GPIO9)
- new net: D1.1 (K), R9.2
Other:
- moved on the sheet: C19

Commit message: Add the initial version of 16bit
Parts:
- added C1, C5: 0.1uf, Capacitor_SMD:C_0402_1005Metric, symbol Device:C
- added C21: 100uf, Capacitor_SMD:C_1206_3216Metric, symbol Device:C
- added C22, C23: 10nf, Capacitor_SMD:C_0402_1005Metric, symbol Device:C
- added R10, R12, R15, R16: 100k, Resistor_SMD:R_0402_1005Metric, symbol Device:R
- added R17, R18: 10k, Resistor_SMD:R_0402_1005Metric, symbol Device:R
- added RV1, RV2: 1M, BreadModular_Pots:Potentiometer_RV09, symbol Device:R_Potentiometer
- added U3: MCP6002-xSN, Package_SO:SOIC-8-1EP_3.9x4.9mm_P1.27mm_EP2.29x3mm, symbol Amplifier_Operational:MCP6002-xSN
- added U4: PT8211, Package_SO:SOIC-8-1EP_3.9x4.9mm_P1.27mm_EP2.29x3mm, symbol Audio:PT8211
- J1, J2: footprint Connector_PinSocket_2.54mm:PinSocket_1x08_P2.54mm_Vertical -> Connector_PinSocket_2.54mm:PinSocket_1x05_P2.54mm_Vertical; symbol Connector:Conn_01x08_Socket -> Connector:Conn_01x05_Socket
- SW1: value SW_SPST -> K2-1808SN-A4SW-01
Connections:
- net +3V3: now also C1.1, C21.1, C5.1, R10.1, R12.1, U3.8 (V+), U4.5 (VDD)
- net GND: now also C1.2, C21.2, C22.1, C23.1, C5.2, R15.2, R16.1, RV1.1, RV2.1, U3.4 (V-), U4.4 (GND)
- net RUN: no longer J2.6 (Pin_6)
- net GOUT_2: now reaches U1.31 (GPIO19)
- net GOUT_2: now also J2.5 (Pin_5)
- net GOUT_1: now reaches U1.32 (GPIO20)
- net GOUT_1: now also J2.4 (Pin_4)
- net GPIO0 renamed BCK
- net BCK: now also U4.1 (BCK); no longer J1.1 (Pin_1)
- net GPIO1 renamed AIN_1
- net AIN_1: now also U1.40 (GPIO26_ADC0), R16.2; no longer U1.3 (GPIO1)
- net GPIO2 renamed AIN_2
- net AIN_2: now also U1.41 (GPIO27_ADC1), R15.1; no longer U1.4 (GPIO2)
- net GPIO25: no longer names the net of U1.37 (GPIO25)
- net GPIO25: no longer J2.5 (Pin_5)
- removed net GPIO26_ADC0: J2.4 (Pin_4), U1.40 (GPIO26_ADC0)
- net GPIO27_ADC1 renamed AOUT_2
- net AOUT_2: now also C23.2, R18.1; no longer U1.41 (GPIO27_ADC1)
- net GPIO28_ADC2 renamed AOUT_1
- net AOUT_1: now also C22.2, R17.1; no longer U1.42 (GPIO28_ADC2)
- net GPIO29_ADC3 renamed BUFF_CV2
- net BUFF_CV2: now also RV2.2; no longer J2.1 (Pin_1)
- net GPIO3: no longer names the net of U1.5 (GPIO3)
- net GPIO3: no longer J1.4 (Pin_4)
- net GPIO4 renamed CV2
- net CV2: now also R12.2, U3.5 (+); no longer U1.7 (GPIO4)
- net GPIO5 renamed MIDI_IN
- net MIDI_IN: now also J1.1 (Pin_1); no longer J1.6 (Pin_6)
- net GPIO6: no longer names the net of U1.9 (GPIO6)
- net GPIO6: no longer J1.7 (Pin_7)
- net GPIO7: no longer names the net of U1.10 (GPIO7)
- net GPIO7: no longer J1.8 (Pin_8)
- net SWCLK: no longer names the net of U1.24 (SWCLK)
- net SWCLK: no longer J2.8 (Pin_8)
- net SWD: no longer names the net of U1.25 (SWD)
- net SWD: no longer J2.7 (Pin_7)
- new net: RV2.3, U3.6 (-), U3.7
- new net: R17.2, U4.6 (L)
- new net: RV1.3, U3.1, U3.2 (-)
- new net: R18.2, U4.8 (R)
- new net BUFF_CV1: RV1.2, U1.42 (GPIO28_ADC2)
- new net CV1: J1.4 (Pin_4), R10.2, U3.3 (+)
- new net DIN: U1.4 (GPIO2), U4.3 (DIN)
- new net MIDI_OUT: J2.1 (Pin_1), U1.7 (GPIO4)
- new net WS: U1.3 (GPIO1), U4.2 (WS)
Other:
- note added: "## CV_IN For this specific chip we don't need the R1 (10k), but for other chips, we may need to use it."
- note added: "## DAC 16-bit PT8211 DAC."
- moved on the sheet: C19, C3, C4, GND1, R2, V_SUPPLY1, Y1
