File: modules/line_in/line_in.kicad_pcb (KiCad board)
At the start: 2 copper layers, 30.5 x 68.6 mm, 28 parts, among them J1 AudioJack3, U1 MCP6002-xSN, U2 MCP6002-xSN, U3 MCP6002-xSN

Commit message: line_in_1.0.0
Other:
- board text added: "LINE_IN 1.0.0"
- board text removed: "LINE_IN 0.2.0"
Changed lines of the file:
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@@
 		(tags "resistor")
 		(property "Reference" "R11"
-			(at 0 -1.17 360)
+			(at 0 -1.17 0)
 			(layer "F.SilkS")
 			(effects
@@
 		)
 		(property "Value" "1k"
-			(at 0 1.17 360)
+			(at 0 1.17 0)
 			(layer "F.Fab")
 			(effects
@@
 		)
 		(fp_text user "${REFERENCE}"
-			(at 0 0 360)
+			(at 0 0 0)
 			(layer "F.Fab")
 			(effects
@@
 		(tags "SOIC SO")
 		(property "Reference" "U3"
-			(at 4.761 1.778 360)
+			(at 4.761 1.778 0)
 			(layer "F.SilkS")
 			(effects
@@
 		(tags "capacitor")
 		(property "Reference" "C5"
-			(at 0 -1.016 360)
+			(at 0 -1.016 0)
 			(layer "F.SilkS")
 			(effects
@@
 		)
 		(property "Value" "0.1uf"
-			(at 0 1.27 360)
+			(at 0 1.27 0)
 			(layer "F.Fab")
 			(effects
@@
 		)
 		(fp_text user "${REFERENCE}"
-			(at 0 0 360)
+			(at 0 0 0)
 			(layer "F.Fab")
 			(effects
@@
 		)
 	)
-	(gr_text "LINE_IN\n0.2.0"
+	(gr_text "LINE_IN\n1.0.0"
 		(at 76.327 107.95 0)
 		(layer "F.SilkS")

Commit message: line_in: update footprints of pots
Parts:
- moved RV2 7.58 mm to (70.3, 73.5), turned to 0 degrees
- moved RV1 7.35 mm to (54.4, 73.5), turned to 0 degrees
Routing:
- net Net-(C2-Pad1): track 8.81 -> 10.3 mm
Other:
- board text added: "LINE_IN 1.0.1"
- board text removed: "LINE_IN 1.0.0"
