File: modules/noise/noise.kicad_pcb (KiCad board)
At the start: 2 copper layers, 30.5 x 68.6 mm, 24 parts, among them U1 ATtiny1616-M, U2 MCP6002-xSN, U3 MCP6002-xSN

Commit message: noise: Add CC:74 label to the tone
Other:
- board text added: "NOISE 0.2.0"
- board text added: "TONE (CC:74)"
- board text removed: "NOISE 0.1.0"
- board text removed: "TONE"
Changed lines of the file:
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@@
 		(tags "resistor")
 		(property "Reference" "R7"
-			(at -1.651 0 360)
+			(at -1.651 0 0)
 			(layer "F.SilkS")
 			(effects
@@
 		)
 		(property "Value" "1k"
-			(at 0 1.17 360)
+			(at 0 1.17 0)
 			(layer "F.Fab")
 			(effects
@@
 		)
 		(fp_text user "${REFERENCE}"
-			(at 0 0 360)
+			(at 0 0 0)
 			(layer "F.Fab")
 			(effects
@@
 		(tags "SOIC SO")
 		(property "Reference" "U2"
-			(at 4.445 -1.905 360)
+			(at 4.445 -1.905 0)
 			(layer "F.SilkS")
 			(effects
@@
 		(tags "resistor")
 		(property "Reference" "R1"
-			(at -1.653 0 360)
+			(at -1.653 0 0)
 			(layer "F.SilkS")
 			(effects
@@
 		)
 		(property "Value" "4.7k"
-			(at 0 1.17 360)
+			(at 0 1.17 0)
 			(layer "F.Fab")
 			(effects
@@
 		)
 		(fp_text user "${REFERENCE}"
-			(at 0 0 360)
+			(at 0 0 0)
 			(layer "F.Fab")
 			(effects
@@
 		(tags "capacitor")
 		(property "Reference" "C2"
-			(at 0 -1.016 360)
+			(at 0 -1.016 0)
 			(layer "F.SilkS")
 			(effects
@@
 		)
 		(property "Value" "100pf"
-			(at 0 1.27 360)
+			(at 0 1.27 0)
 			(layer "F.Fab")
 			(effects
@@
 		)
 		(fp_text user "${REFERENCE}"
-			(at 0 0 360)
+			(at 0 0 0)
 			(layer "F.Fab")
 			(effects
@@
 		(tags "resistor")
 		(property "Reference" "R6"
-			(at -1.649 0 360)
+			(at -1.649 0 0)
 			(layer "F.SilkS")
 			(effects
@@
 		)
 		(property "Value" "330"
-			(at 0 1.17 360)
+			(at 0 1.17 0)
 			(layer "F.Fab")
 			(effects
@@
 		)
 		(fp_text user "${REFERENCE}"
-			(at 0 0 360)
+			(at 0 0 0)
 			(layer "F.Fab")
 			(effects
@@
 		(tags "resistor")
 		(property "Reference" "R8"
-			(at -1.778 0 360)
+			(at -1.778 0 0)
 			(layer "F.SilkS")
 			(effects
@@
 		)
 		(property "Value" "22k"
-			(at 0 1.17 360)
+			(at 0 1.17 0)
 			(layer "F.Fab")
 			(effects
@@
 		)
 		(fp_text user "${REFERENCE}"
-			(at 0 0 360)
+			(at 0 0 0)
 			(layer "F.Fab")
 			(effects
@@
 		(tags "SOIC SO")
 		(property "Reference" "U3"
-			(at 4.507 -1.536 360)
+			(at 4.507 -1.536 0)
 			(layer "F.SilkS")
 			(effects
@@
 		)
 	)
-	(gr_text "NOISE\n0.1.0"
+	(gr_text "NOISE\n0.2.0"
 		(at 76.327 107.95 0)
 		(layer "F.SilkS")
@@
 		)
 	)
-	(gr_text "TONE"
-		(at 60.325 76.835 0)
+	(gr_text "TONE (CC:74)"
+		(at 62.3 76.5 0)
 		(layer "F.SilkS")
 		(effects
@@
 				(thickness 0.15)
 			)
-			(justify left bottom)
+			(justify bottom)
 		)
 	)

Commit message: noise: add MIDI Thru support
Connections:
- OUTPUT1 pad 1: WHITE_NOISE -> MIDI
- OUTPUT1 pad 3: BLUE_NOISE -> WHITE_NOISE
Routing:
- net MIDI: track 28.6 -> 49.7 mm
- net BLUE_NOISE: track 58.5 -> 52.8 mm
- net WHITE_NOISE: track 51.6 -> 49.1 mm
Other:
- board text added: "NOISE 0.3.0"
- board text removed: "NOISE 0.2.0"
Changed lines of the file:
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@@
 			(layers "*.Cu" "*.Mask")
 			(remove_unused_layers no)
-			(net 14 "WHITE_NOISE")
+			(net 10 "MIDI")
 			(pinfunction "Pin_1")
 			(pintype "passive")
@@
 			(layers "*.Cu" "*.Mask")
 			(remove_unused_layers no)
-			(net 13 "BLUE_NOISE")
+			(net 14 "WHITE_NOISE")
 			(pinfunction "Pin_3")
 			(pintype "passive")
@@
 		)
 	)
-	(gr_text "NOISE\n0.2.0"
+	(gr_text "NOISE\n0.3.0"
 		(at 76.327 107.95 0)
 		(layer "F.SilkS")
@@
 		)
 	)
-	(gr_text "BLUE"
+	(gr_text "WHITE"
 		(at 71.755 51.435 0)
 		(layer "F.SilkS")
@@
 		)
 	)
-	(gr_text "WHITE"
+	(gr_text "MIDI"
 		(at 71.755 46.355 0)
 		(layer "F.SilkS")
@@
 	)
 	(segment
+		(start 50.8 45.72)
+		(end 52.832 45.72)
+		(width 0.15)
+		(layer "F.Cu")
+		(net 10)
+	)
+	(segment
 		(start 66.263 53.576025)
 		(end 66.263 57.95498)
@@
 	)
 	(segment
+		(start 73.66 45.72)
+		(end 73.29 46.09)
+		(width 0.15)
+		(layer "F.Cu")
+		(net 10)
+	)
+	(segment
 		(start 66.263 57.95498)
 		(end 65.71598 58.502)
@@
 	)
 	(segment
-		(start 50.8 45.72)
+		(start 53.202 46.09)
+		(end 52.832 45.72)
+		(width 0.15)
+		(layer "F.Cu")
+		(net 10)
+	)
+	(segment
+		(start 73.29 46.09)
+		(end 53.202 46.09)
+		(width 0.15)
+		(layer "F.Cu")
+		(net 10)
+	)
+	(segment
+		(start 52.832 45.72)
 		(end 52.959 45.72)
 		(width 0.15)
@@
 	)
 	(segment
-		(start 76.327 51.181)
-		(end 75.946 50.8)
-		(width 0.15)
-		(layer "F.Cu")
-		(net 13)
-	)
-	(segment
 		(start 75.678974 76.962)
 		(end 76.327 76.313974)
@@
 	)
 	(segment
-		(start 73.66 50.8)
-		(end 73.66 53.34)
-		(width 0.15)
-		(layer "F.Cu")
-		(net 13)
-	)
-	(segment
 		(start 54.991 73.152)
 		(end 54.991 76.2)
@@
 	)
 	(segment
-		(start 75.946 50.8)
-		(end 73.66 50.8)
-		(width 0.15)
-		(layer "F.Cu")
-		(net 13)
-	)
-	(segment
 		(start 76.327 76.313974)
-		(end 76.327 51.181)
+		(end 76.327 54.737)
 		(width 0.15)
 		(layer "F.Cu")
@@
 		(start 51.947 73.152)
 		(end 53.467 73.152)
+		(width 0.15)
+		(layer "F.Cu")
+		(net 13)
+	)
+	(segment
+		(start 73.66 53.34)
+		(end 74.93 53.34)
+		(width 0.15)
+		(layer "F.Cu")
+		(net 13)
+	)
+	(segment
+		(start 74.93 53.34)
+		(end 76.327 54.737)
 		(width 0.15)
 		(layer "F.Cu")
@@
 	)
 	(segment
+		(start 73.66 48.26)
+		(end 71.247 48.26)
+		(width 0.15)
+		(layer "F.Cu")
+		(net 14)
+	)
+	(segment
 		(start 66.888 56.22)
 		(end 67.056 56.388)
@@
 	)
 	(segment
-		(start 68.961 48.133)
-		(end 71.374 45.72)
-		(width 0.15)
-		(layer "F.Cu")
-		(net 14)
-	)
-	(segment
-		(start 73.66 48.26)
-		(end 73.66 45.72)
+		(start 68.961 53.848)
+		(end 68.961 50.546)
 		(width 0.15)
 		(layer "F.Cu")
@@
 	)
 	(segment
+		(start 71.247 48.26)
+		(end 68.961 50.546)
+		(width 0.15)
+		(layer "F.Cu")
+		(net 14)
+	)
+	(segment
 		(start 67.056 56.388)
 		(end 67.056 55.753)
@@
 	)
 	(segment
-		(start 68.961 53.848)
-		(end 68.961 48.133)
-		(width 0.15)
-		(layer "F.Cu")
-		(net 14)
-	)
-	(segment
 		(start 72.505 64.9)
 		(end 72.505 61.837)
@@
 	)
 	(segment
+		(start 73.66 48.26)
+		(end 73.66 50.8)
+		(width 0.15)
+		(layer "F.Cu")
+		(net 14)
+	)
+	(segment
 		(start 51.816 60.579)
 		(end 52.07 60.325)
 		(width 0.15)
 		(layer "F.Cu")
-		(net 14)
-	)
-	(segment
-		(start 71.374 45.72)
-		(end 73.66 45.72)
-		(width 0.15)
-		(layer "F.Cu")

Commit message: noise_1.0.0
Other:
- board text added: "NOISE 1.0.0"
- board text removed: "NOISE 0.3.0"
Changed lines of the file:
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@@
 		)
 	)
-	(gr_text "NOISE\n0.3.0"
+	(gr_text "NOISE\n1.0.0"
 		(at 76.327 107.95 0)
 		(layer "F.SilkS")

Commit message: noise: update footprints of pots
Parts:
- moved RV2 7.69 mm to (55.0, 83.7), turned to 0 degrees
- moved RV3 7.48 mm to (69.6, 83.7), turned to 0 degrees
- moved RV1 7.47 mm to (62.4, 66.7), turned to 0 degrees
- moved R8 0.25 mm to (72.9, 77.5)
Routing:
- net V_MID: track 46.8 -> 47.4 mm
Other:
- board text added: "NOISE 1.0.1"
- board text removed: "NOISE 1.0.0"
