File: modules/wave/wave.kicad_pcb (KiCad board)
At the start: 2 copper layers, 30.5 x 68.6 mm, 33 parts, among them U1 MCP6002-xSN, U2 MCP6002-xSN

Commit message: wave_1.0.0
Other:
- board text added: "WAVE 1.0.0"
- board text removed: "WAVE 0.1.0"
Changed lines of the file:
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@@
 		)
 	)
-	(gr_text "WAVE\n0.1.0"
+	(gr_text "WAVE\n1.0.0"
 		(at 76.327 107.95 0)
 		(layer "F.SilkS")

Commit message: wave: update footprints of pots
Parts:
- RV1: value 50k -> 1M
- RV2: value 1M -> 50k
- moved RV2 7.69 mm to (70.3, 72.3), turned to 0 degrees
- moved RV1 7.48 mm to (54.4, 72.3), turned to 0 degrees
Routing:
- net Net-(RV1-Pad3): track 15.4 -> 16.1 mm
Other:
- board text added: "WAVE 1.0.1"
- board text removed: "WAVE 1.0.0"
