File: modules/16bit/16bit.kicad_sch (KiCad schematic)
At the start: 59 parts, among them J1 Conn_01x08_Socket, J2 Conn_01x08_Socket, J5 USB_C_Receptacle_USB2.0_14P, SW1 K2-1808SN-A4SW-01, SW2 K2-1808SN-A4SW-01, SW3 K2-1808SN-A4SW-01, U1 RP2350_60QFN, U2 W25Q128JVS, U3 MCP6002-xSN, U4 PT8211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

Commit message: Revert "16bit: Add Ditial Audio In & Out support"
This reverts commit 124be004a509aaac87467e57efb917f1b3001793.
Connections:
- net CV2: now reaches R12.2, U3.5 (+)
- net CV2: now also J1.5 (Pin_5)
- net DGITIAL_AUDIO_IN: no longer names the net of U1.12 (GPIO8)
- net DGITIAL_AUDIO_IN: no longer J1.5 (Pin_5)
- net DGITIAL_AUDIO_OUT renamed GOUT_2
Other:
- moved on the sheet: J2
Changed lines of the file:
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@@
 	)
 	(junction
+		(at 43.18 368.3)
+		(diameter 0)
+		(color 0 0 0 0)
+	)
+	(junction
 		(at 214.63 81.28)
 		(diameter 0)
@@
 	(wire
 		(pts
-			(xy 240.03 132.08) (xy 229.87 132.08)
-		)
-		(stroke
-			(width 0)
-			(type default)
-		)
-	)
-	(wire
-		(pts
 			(xy 105.41 322.58) (xy 105.41 321.31)
 		)
@@
 	(wire
 		(pts
-			(xy 83.82 370.84) (xy 83.82 381)
+			(xy 463.55 128.27) (xy 469.9 128.27)
 		)
 		(stroke
@@
 	(wire
 		(pts
-			(xy 229.87 114.3) (xy 240.03 114.3)
+			(xy 83.82 370.84) (xy 83.82 381)
 		)
 		(stroke
@@
 	(wire
 		(pts
-			(xy 266.7 307.34) (xy 279.4 307.34)
+			(xy 229.87 114.3) (xy 240.03 114.3)
 		)
 		(stroke
@@
 	(wire
 		(pts
-			(xy 21.59 266.7) (xy 21.59 269.24)
+			(xy 266.7 307.34) (xy 279.4 307.34)
 		)
 		(stroke
@@
 	(wire
 		(pts
-			(xy 537.21 71.12) (xy 539.75 71.12)
+			(xy 21.59 266.7) (xy 21.59 269.24)
 		)
 		(stroke
@@
 	(wire
 		(pts
-			(xy 40.64 69.85) (xy 40.64 80.01)
+			(xy 537.21 71.12) (xy 539.75 71.12)
 		)
 		(stroke
@@
 	(wire
 		(pts
-			(xy 199.39 93.98) (xy 199.39 81.28)
+			(xy 40.64 69.85) (xy 40.64 80.01)
 		)
 		(stroke
@@
 	(wire
 		(pts
-			(xy 469.9 128.27) (xy 463.55 128.27)
+			(xy 199.39 93.98) (xy 199.39 81.28)
 		)
 		(stroke
@@
 	(wire
 		(pts
+			(xy 502.92 125.73) (xy 508 125.73)
+		)
+		(stroke
+			(width 0)
+			(type default)
+		)
+	)
+	(wire
+		(pts
 			(xy 201.93 93.98) (xy 201.93 81.28)
 		)
@@
 	(wire
 		(pts
-			(xy 525.78 121.92) (xy 530.86 121.92)
+			(xy 502.92 120.65) (xy 508 120.65)
 		)
 		(stroke
@@
 	(wire
 		(pts
+			(xy 33.02 368.3) (xy 43.18 368.3)
+		)
+		(stroke
+			(width 0)
+			(type default)
+		)
+	)
+	(wire
+		(pts
 			(xy 143.51 60.96) (xy 154.94 60.96)
 		)
@@
 	(wire
 		(pts
-			(xy 525.78 119.38) (xy 530.86 119.38)
+			(xy 502.92 118.11) (xy 508 118.11)
 		)
 		(stroke
@@
 	(wire
 		(pts
-			(xy 525.78 127) (xy 530.86 127)
-		)
-		(stroke
-			(width 0)
-			(type default)
-		)
-	)
-	(wire
-		(pts
 			(xy 537.21 212.09) (xy 529.59 212.09)
 		)
@@
 	(wire
 		(pts
-			(xy 525.78 116.84) (xy 530.86 116.84)
+			(xy 502.92 115.57) (xy 508 115.57)
 		)
 		(stroke
@@
 	(wire
 		(pts
-			(xy 525.78 124.46) (xy 530.86 124.46)
+			(xy 502.92 123.19) (xy 508 123.19)
 		)
 		(stroke
@@
 		)
 	)
+	(global_label "CV2"
+		(shape input)
+		(at 469.9 128.27 0)
+		(fields_autoplaced yes)
+		(effects
+			(font
+				(size 1.27 1.27)
+			)
+			(justify left)
+		)
+		(property "Intersheetrefs" "${INTERSHEET_REFS}"
+			(at 475.7991 128.27 0)
+			(effects
+				(font
+					(size 1.27 1.27)
+				)
+				(justify left)
+				(hide yes)
+			)
+		)
+	)
 	(global_label "GOUT_1"
 		(shape output)
@@
 	(global_label "GOUT_1"
 		(shape output)
-		(at 525.78 124.46 180)
+		(at 502.92 123.19 180)
 		(fields_autoplaced yes)
 		(effects
@@
 		)
 		(property "Intersheetrefs" "${INTERSHEET_REFS}"
-			(at 516.3733 124.46 0)
+			(at 493.5133 123.19 0)
 			(effects
 				(font
@@
 	(global_label "MIDI_OUT"
 		(shape output)
-		(at 525.78 116.84 180)
+		(at 502.92 115.57 180)
 		(fields_autoplaced yes)
 		(effects
@@
 		)
 		(property "Intersheetrefs" "${INTERSHEET_REFS}"
-			(at 514.9218 116.84 0)
+			(at 492.0618 115.57 0)
 			(effects
 				(font
@@
 		)
 	)
-	(global_label "DGITIAL_AUDIO_OUT"
+	(global_label "GOUT_2"
 		(shape output)
 		(at 234.95 160.02 0)
@@
 		)
 		(property "Intersheetrefs" "${INTERSHEET_REFS}"
-			(at 255.3031 160.02 0)
-			(effects
-				(font
-					(size 1.27 1.27)
-				)
-				(justify left)
-				(hide yes)
-			)
-		)
-	)
-	(global_label "DGITIAL_AUDIO_IN"
-		(shape input)
-		(at 240.03 132.08 0)
-		(fields_autoplaced yes)
-		(effects
-			(font
-				(size 1.27 1.27)
-			)
-			(justify left)
-		)
-		(property "Intersheetrefs" "${INTERSHEET_REFS}"
-			(at 258.6898 132.08 0)
+			(at 244.3567 160.02 0)
 			(effects
 				(font
@@
 		)
 	)
-	(global_label "DGITIAL_AUDIO_IN"
+	(global_label "AIN_1"
 		(shape input)
-		(at 469.9 128.27 0)
+		(at 469.9 120.65 0)
 		(fields_autoplaced yes)
 		(effects
@@
 		)
 		(property "Intersheetrefs" "${INTERSHEET_REFS}"
-			(at 488.5598 128.27 0)
+			(at 477.432 120.65 0)
 			(effects
 				(font
@@
 		)
 	)
-	(global_label "AIN_1"
+	(global_label "CV2"
 		(shape input)
-		(at 469.9 120.65 0)
+		(at 33.02 368.3 180)
 		(fields_autoplaced yes)
 		(effects
@@
 				(size 1.27 1.27)
 			)
-			(justify left)
+			(justify right)
 		)
 		(property "Intersheetrefs" "${INTERSHEET_REFS}"
-			(at 477.432 120.65 0)
+			(at 26.4667 368.3 0)
 			(effects
 				(font
 					(size 1.27 1.27)
 				)
-				(justify left)
+				(justify right)
 				(hide yes)
 			)
@@
 	(global_label "AOUT_1"
 		(shape output)
-		(at 525.78 119.38 180)
+		(at 502.92 118.11 180)
 		(fields_autoplaced yes)
 		(effects
@@
 		)
 		(property "Intersheetrefs" "${INTERSHEET_REFS}"
-			(at 516.5547 119.38 0)
+			(at 493.6947 118.11 0)
 			(effects
 				(font
@@
 		)
 	)
+	(global_label "GOUT_2"
+		(shape output)
+		(at 502.92 125.73 180)
+		(fields_autoplaced yes)
+		(effects
+			(font
+				(size 1.27 1.27)
+			)
+			(justify right)
+		)
+		(property "Intersheetrefs" "${INTERSHEET_REFS}"
+			(at 493.5133 125.73 0)
+			(effects
+				(font
+					(size 1.27 1.27)
+				)
+				(justify right)
+				(hide yes)
+			)
+		)
+	)
 	(global_label "USB_D-"
 		(shape bidirectional)
@@
 	(global_label "AOUT_2"
 		(shape output)
-		(at 525.78 121.92 180)
+		(at 502.92 120.65 180)
 		(fields_autoplaced yes)
 		(effects
@@
 		)
 		(property "Intersheetrefs" "${INTERSHEET_REFS}"
-			(at 516.5547 121.92 0)
+			(at 493.6947 120.65 0)
 			(effects
 				(font
@@
 		)
 	)
-	(global_label "DGITIAL_AUDIO_OUT"
-		(shape output)
-		(at 525.78 127 180)
-		(fields_autoplaced yes)
-		(effects
-			(font
-				(size 1.27 1.27)
-			)
-			(justify right)
-		)
-		(property "Intersheetrefs" "${INTERSHEET_REFS}"
-			(at 505.4269 127 0)
-			(effects
-				(font
-					(size 1.27 1.27)
-				)
-				(justify right)
-				(hide yes)
-			)
-		)
-	)
 	(symbol
 		(lib_id "power:+3V3")
@@
 	(symbol
 		(lib_id "Connector:Conn_01x05_Socket")
-		(at 535.94 121.92 0)
+		(at 513.08 120.65 0)
 		(unit 1)
 		(exclude_from_sim no)
@@
 		(dnp no)
 		(property "Reference" "J2"
-			(at 537.21 120.904 90)
+			(at 514.35 119.634 90)
 			(effects
 				(font
@@
 		)
 		(property "Value" "Conn_01x08_Socket"
-			(at 539.242 121.412 90)
+			(at 516.382 120.142 90)
 			(effects
 				(font
@@
 		)
 		(property "Footprint" "Connector_PinSocket_2.54mm:PinSocket_1x05_P2.54mm_Vertical"
-			(at 535.94 121.92 0)
+			(at 513.08 120.65 0)
 			(effects
 				(font
@@
 		)
 		(property "Datasheet" "~"
-			(at 535.94 121.92 0)
+			(at 513.08 120.65 0)
 			(effects
 				(font
@@
 		)
 		(property "Description" "Generic connector, single row, 01x05, script generated"
-			(at 535.94 121.92 0)
+			(at 513.08 120.65 0)
 			(effects
 				(font
