File: modules/mcc/mcc.kicad_pcb (KiCad board)
At the start: 2 copper layers, 30.5 x 68.6 mm, 22 parts, among them SW1 K2-1808SN-A4SW-01, U1 ATtiny1616-M

Commit message: mcc_1.0.0
Other:
- board text added: "MCC 1.0.0"
- board text removed: "MCC 0.1.0"
Changed lines of the file:
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@@
 		)
 	)
-	(gr_text "MCC\n0.1.0"
+	(gr_text "MCC\n1.0.0"
 		(at 76.327 107.95 0)
 		(layer "F.SilkS")
