File: modules/4mix/sends.kicad_sch (KiCad schematic)
At the start: 4 parts

Commit message: Fix phase issues & cascading support. * There were some phase issues related when mixing returns   in the master mixer. * Now input and mixout has the same phase * Add in_mixout, in_send_a & in_send_b to cascase another mixser
Parts:
- renumbered R35 to R51, R36 to R52
Changed lines of the file:
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@@
 		(dnp no)
 		(fields_autoplaced yes)
-		(property "Reference" "R36"
+		(property "Reference" "R52"
 			(at 97.79 113.03 90)
 			(effects
@@
 			(project "4mix"
 				(path "/b63493d3-5f6d-47e3-845b-87e7090fc1ab/074c6592-d8f2-41b8-8f7b-9cda7a97378a"
-					(reference "R36")
+					(reference "R52")
 					(unit 1)
 				)
 				(path "/b63493d3-5f6d-47e3-845b-87e7090fc1ab/1ae334da-fe90-433f-a798-500782e5ff21"
-					(reference "R38")
+					(reference "R54")
 					(unit 1)
 				)
 				(path "/b63493d3-5f6d-47e3-845b-87e7090fc1ab/24708e82-002c-49b4-ad8d-d7b04b998c06"
-					(reference "R34")
+					(reference "R50")
 					(unit 1)
 				)
 				(path "/b63493d3-5f6d-47e3-845b-87e7090fc1ab/393550cb-40c9-4351-a1f3-230233b59078"
-					(reference "R32")
+					(reference "R48")
 					(unit 1)
 				)
@@
 		(dnp no)
 		(fields_autoplaced yes)
-		(property "Reference" "R35"
+		(property "Reference" "R51"
 			(at 97.79 81.28 90)
 			(effects
@@
 			(project "4mix"
 				(path "/b63493d3-5f6d-47e3-845b-87e7090fc1ab/074c6592-d8f2-41b8-8f7b-9cda7a97378a"
-					(reference "R35")
+					(reference "R51")
 					(unit 1)
 				)
 				(path "/b63493d3-5f6d-47e3-845b-87e7090fc1ab/1ae334da-fe90-433f-a798-500782e5ff21"
-					(reference "R37")
+					(reference "R53")
 					(unit 1)
 				)
 				(path "/b63493d3-5f6d-47e3-845b-87e7090fc1ab/24708e82-002c-49b4-ad8d-d7b04b998c06"
-					(reference "R33")
+					(reference "R49")
 					(unit 1)
 				)
 				(path "/b63493d3-5f6d-47e3-845b-87e7090fc1ab/393550cb-40c9-4351-a1f3-230233b59078"
-					(reference "R31")
+					(reference "R47")
 					(unit 1)
 				)

Commit message: Add some improvements to 4mix
Parts:
- renumbered R51 to R49, R52 to R50, RV12 to RV10, RV13 to RV11
Changed lines of the file:
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@@
 (kicad_sch
-	(version 20231120)
+	(version 20250114)
 	(generator "eeschema")
-	(generator_version "8.0")
+	(generator_version "9.0")
 	(paper "A4")
 	(junction
@@
 		(dnp no)
 		(fields_autoplaced yes)
-		(property "Reference" "R52"
+		(property "Reference" "R50"
 			(at 97.79 113.03 90)
 			(effects
@@
 				(path "/b63493d3-5f6d-47e3-845b-87e7090fc1ab/24708e82-002c-49b4-ad8d-d7b04b998c06"
 					(reference "R50")
-					(unit 1)
-				)
-				(path "/b63493d3-5f6d-47e3-845b-87e7090fc1ab/393550cb-40c9-4351-a1f3-230233b59078"
-					(reference "R48")
 					(unit 1)
 				)
@@
 		(dnp no)
 		(fields_autoplaced yes)
-		(property "Reference" "R51"
+		(property "Reference" "R49"
 			(at 97.79 81.28 90)
 			(effects
@@
 				(path "/b63493d3-5f6d-47e3-845b-87e7090fc1ab/24708e82-002c-49b4-ad8d-d7b04b998c06"
 					(reference "R49")
-					(unit 1)
-				)
-				(path "/b63493d3-5f6d-47e3-845b-87e7090fc1ab/393550cb-40c9-4351-a1f3-230233b59078"
-					(reference "R47")
 					(unit 1)
 				)
@@
 		(on_board yes)
 		(dnp no)
-		(property "Reference" "RV13"
+		(property "Reference" "RV11"
 			(at 78.74 104.902 90)
 			(effects
@@
 				(path "/b63493d3-5f6d-47e3-845b-87e7090fc1ab/24708e82-002c-49b4-ad8d-d7b04b998c06"
 					(reference "RV11")
-					(unit 1)
-				)
-				(path "/b63493d3-5f6d-47e3-845b-87e7090fc1ab/393550cb-40c9-4351-a1f3-230233b59078"
-					(reference "RV9")
 					(unit 1)
 				)
@@
 		(on_board yes)
 		(dnp no)
-		(property "Reference" "RV12"
+		(property "Reference" "RV10"
 			(at 78.74 73.152 90)
 			(effects
@@
 					(unit 1)
 				)
-				(path "/b63493d3-5f6d-47e3-845b-87e7090fc1ab/393550cb-40c9-4351-a1f3-230233b59078"
-					(reference "RV8")
-					(unit 1)
-				)
