File: modules/4mix/channel.kicad_sch (KiCad schematic)
At the start: 21 parts, among them U9 MCP6002-xSN

Commit message: Finished the new schematic for 4mix
Parts:
- removed C10, C12: 0.1uf, Capacitor_SMD:C_0402_1005Metric, symbol Device:C
- removed C11: 10uf, Capacitor_SMD:C_0402_1005Metric, symbol Device:C
- removed C13: 47pf, Capacitor_SMD:C_0402_1005Metric, symbol Device:C
- removed R47: 1M, Resistor_SMD:R_0402_1005Metric, symbol Device:R
- removed R48, R63, R65, R66, R67: 56k, Resistor_SMD:R_0402_1005Metric, symbol Device:R
- removed R64, R68, R69, R70, R71, R72, R73: 100, Resistor_SMD:R_0402_1005Metric, symbol Device:R
- removed RV20, RV8, RV9: 50k, BreadModular_Pots:Potentiometer_RV09, symbol Device:R_Potentiometer
- removed U9: MCP6002-xSN, Package_SO:SOIC-8-1EP_3.9x4.9mm_P1.27mm_EP2.29x3mm, symbol Amplifier_Operational:MCP6002-xSN
Other:
- note removed: "This should place at the summing opamp"
