File: modules/4mix/overdrive.kicad_sch (KiCad schematic)
At the start: 14 parts, among them U6 MCP6002-xSN

Commit message: Fix phase issues & cascading support. * There were some phase issues related when mixing returns   in the master mixer. * Now input and mixout has the same phase * Add in_mixout, in_send_a & in_send_b to cascase another mixser
Parts:
- renumbered C7 to C9, D3 to D2, D5 to D3, D6 to D4, R30 to R55, R44 to R56, R45 to R57, R46 to R58, R47 to R59, R48 to R60, U6 to U8
Changed lines of the file:
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@@
 		(dnp no)
 		(fields_autoplaced yes)
-		(property "Reference" "U6"
+		(property "Reference" "U8"
 			(at 77.47 49.53 0)
 			(effects
@@
 			(project "4mix"
 				(path "/b63493d3-5f6d-47e3-845b-87e7090fc1ab/d0b612c1-0c25-4058-bf92-38ae27a09cef"
-					(reference "U6")
+					(reference "U8")
 					(unit 1)
 				)
@@
 		(on_board yes)
 		(dnp no)
-		(property "Reference" "#PWR022"
+		(property "Reference" "#PWR027"
 			(at 251.46 80.01 0)
 			(effects
@@
 			(project "4mix"
 				(path "/b63493d3-5f6d-47e3-845b-87e7090fc1ab/d0b612c1-0c25-4058-bf92-38ae27a09cef"
-					(reference "#PWR022")
+					(reference "#PWR027")
 					(unit 1)
 				)
@@
 		(dnp no)
 		(fields_autoplaced yes)
-		(property "Reference" "C7"
+		(property "Reference" "C9"
 			(at 264.16 85.0899 0)
 			(effects
@@
 			(project "4mix"
 				(path "/b63493d3-5f6d-47e3-845b-87e7090fc1ab/d0b612c1-0c25-4058-bf92-38ae27a09cef"
-					(reference "C7")
+					(reference "C9")
 					(unit 1)
 				)
@@
 		(dnp no)
 		(fields_autoplaced yes)
-		(property "Reference" "U6"
+		(property "Reference" "U8"
 			(at 132.08 50.8 0)
 			(effects
@@
 			(project "4mix"
 				(path "/b63493d3-5f6d-47e3-845b-87e7090fc1ab/d0b612c1-0c25-4058-bf92-38ae27a09cef"
-					(reference "U6")
+					(reference "U8")
 					(unit 2)
 				)
@@
 		(dnp no)
 		(fields_autoplaced yes)
-		(property "Reference" "R47"
+		(property "Reference" "R59"
 			(at 166.37 41.91 90)
 			(effects
@@
 			(project "4mix"
 				(path "/b63493d3-5f6d-47e3-845b-87e7090fc1ab/d0b612c1-0c25-4058-bf92-38ae27a09cef"
-					(reference "R47")
+					(reference "R59")
 					(unit 1)
 				)
@@
 		(dnp no)
 		(fields_autoplaced yes)
-		(property "Reference" "R48"
+		(property "Reference" "R60"
 			(at 181.61 60.96 90)
 			(effects
@@
 			(project "4mix"
 				(path "/b63493d3-5f6d-47e3-845b-87e7090fc1ab/d0b612c1-0c25-4058-bf92-38ae27a09cef"
-					(reference "R48")
+					(reference "R60")
 					(unit 1)
 				)
@@
 		(dnp no)
 		(fields_autoplaced yes)
-		(property "Reference" "D3"
+		(property "Reference" "D2"
 			(at 135.5725 82.55 0)
 			(effects
@@
 			(project "4mix"
 				(path "/b63493d3-5f6d-47e3-845b-87e7090fc1ab/d0b612c1-0c25-4058-bf92-38ae27a09cef"
-					(reference "D3")
+					(reference "D2")
 					(unit 1)
 				)
@@
 		(on_board yes)
 		(dnp no)
-		(property "Reference" "R46"
+		(property "Reference" "R58"
 			(at 132.08 70.104 90)
 			(effects
@@
 			(project "4mix"
 				(path "/b63493d3-5f6d-47e3-845b-87e7090fc1ab/d0b612c1-0c25-4058-bf92-38ae27a09cef"
-					(reference "R46")
+					(reference "R58")
 					(unit 1)
 				)
@@
 		(dnp no)
 		(fields_autoplaced yes)
-		(property "Reference" "R45"
+		(property "Reference" "R57"
 			(at 115.57 57.15 90)
 			(effects
@@
 			(project "4mix"
 				(path "/b63493d3-5f6d-47e3-845b-87e7090fc1ab/d0b612c1-0c25-4058-bf92-38ae27a09cef"
-					(reference "R45")
+					(reference "R57")
 					(unit 1)
 				)
@@
 		(on_board yes)
 		(dnp no)
-		(property "Reference" "#PWR023"
+		(property "Reference" "#PWR028"
 			(at 251.46 102.87 0)
 			(effects
@@
 			(project "4mix"
 				(path "/b63493d3-5f6d-47e3-845b-87e7090fc1ab/d0b612c1-0c25-4058-bf92-38ae27a09cef"
-					(reference "#PWR023")
+					(reference "#PWR028")
 					(unit 1)
 				)
@@
 		(dnp no)
 		(fields_autoplaced yes)
-		(property "Reference" "R30"
+		(property "Reference" "R55"
 			(at 59.69 55.88 90)
 			(effects
@@
 			(project "4mix"
 				(path "/b63493d3-5f6d-47e3-845b-87e7090fc1ab/d0b612c1-0c25-4058-bf92-38ae27a09cef"
-					(reference "R30")
+					(reference "R55")
 					(unit 1)
 				)
@@
 		(dnp no)
 		(fields_autoplaced yes)
-		(property "Reference" "D6"
+		(property "Reference" "D4"
 			(at 166.0525 66.04 0)
 			(effects
@@
 			(project "4mix"
 				(path "/b63493d3-5f6d-47e3-845b-87e7090fc1ab/d0b612c1-0c25-4058-bf92-38ae27a09cef"
-					(reference "D6")
+					(reference "D4")
 					(unit 1)
 				)
@@
 		(on_board yes)
 		(dnp no)
-		(property "Reference" "U6"
+		(property "Reference" "U8"
 			(at 243.332 93.218 90)
 			(effects
@@
 			(project "4mix"
 				(path "/b63493d3-5f6d-47e3-845b-87e7090fc1ab/d0b612c1-0c25-4058-bf92-38ae27a09cef"
-					(reference "U6")
+					(reference "U8")
 					(unit 3)
 				)
@@
 		(dnp no)
 		(fields_autoplaced yes)
-		(property "Reference" "R44"
+		(property "Reference" "R56"
 			(at 77.47 67.31 90)
 			(effects
@@
 			(project "4mix"
 				(path "/b63493d3-5f6d-47e3-845b-87e7090fc1ab/d0b612c1-0c25-4058-bf92-38ae27a09cef"
-					(reference "R44")
+					(reference "R56")
 					(unit 1)
 				)
@@
 		(dnp no)
 		(fields_autoplaced yes)
-		(property "Reference" "D5"
+		(property "Reference" "D3"
 			(at 166.6875 54.61 0)
 			(effects
@@
 			(project "4mix"
 				(path "/b63493d3-5f6d-47e3-845b-87e7090fc1ab/d0b612c1-0c25-4058-bf92-38ae27a09cef"
-					(reference "D5")
-					(unit 1)
-				)
+					(reference "D3")
+					(unit 1)
+				)

Commit message: Finished the new schematic for 4mix
Parts:
- renumbered C9 to C35, R55 to R90, R56 to R91, R57 to R92, R58 to R93, R59 to R94, R60 to R95, U8 to U11
Changed lines of the file:
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@@
 		(dnp no)
 		(fields_autoplaced yes)
-		(property "Reference" "U8"
+		(property "Reference" "U11"
 			(at 77.47 49.53 0)
 			(effects
@@
 			(project "4mix"
 				(path "/b63493d3-5f6d-47e3-845b-87e7090fc1ab/d0b612c1-0c25-4058-bf92-38ae27a09cef"
-					(reference "U8")
+					(reference "U11")
 					(unit 1)
 				)
@@
 		(on_board yes)
 		(dnp no)
-		(property "Reference" "#PWR027"
+		(property "Reference" "#PWR037"
 			(at 251.46 80.01 0)
 			(effects
@@
 			(project "4mix"
 				(path "/b63493d3-5f6d-47e3-845b-87e7090fc1ab/d0b612c1-0c25-4058-bf92-38ae27a09cef"
-					(reference "#PWR027")
+					(reference "#PWR037")
 					(unit 1)
 				)
@@
 		(dnp no)
 		(fields_autoplaced yes)
-		(property "Reference" "C9"
+		(property "Reference" "C35"
 			(at 264.16 85.0899 0)
 			(effects
@@
 			(project "4mix"
 				(path "/b63493d3-5f6d-47e3-845b-87e7090fc1ab/d0b612c1-0c25-4058-bf92-38ae27a09cef"
-					(reference "C9")
+					(reference "C35")
 					(unit 1)
 				)
@@
 		(dnp no)
 		(fields_autoplaced yes)
-		(property "Reference" "U8"
+		(property "Reference" "U11"
 			(at 132.08 50.8 0)
 			(effects
@@
 			(project "4mix"
 				(path "/b63493d3-5f6d-47e3-845b-87e7090fc1ab/d0b612c1-0c25-4058-bf92-38ae27a09cef"
-					(reference "U8")
+					(reference "U11")
 					(unit 2)
 				)
@@
 		(dnp no)
 		(fields_autoplaced yes)
-		(property "Reference" "R59"
+		(property "Reference" "R94"
 			(at 166.37 41.91 90)
 			(effects
@@
 			(project "4mix"
 				(path "/b63493d3-5f6d-47e3-845b-87e7090fc1ab/d0b612c1-0c25-4058-bf92-38ae27a09cef"
-					(reference "R59")
+					(reference "R94")
 					(unit 1)
 				)
@@
 		(dnp no)
 		(fields_autoplaced yes)
-		(property "Reference" "R60"
+		(property "Reference" "R95"
 			(at 181.61 60.96 90)
 			(effects
@@
 			(project "4mix"
 				(path "/b63493d3-5f6d-47e3-845b-87e7090fc1ab/d0b612c1-0c25-4058-bf92-38ae27a09cef"
-					(reference "R60")
+					(reference "R95")
 					(unit 1)
 				)
@@
 		(on_board yes)
 		(dnp no)
-		(property "Reference" "R58"
+		(property "Reference" "R93"
 			(at 132.08 70.104 90)
 			(effects
@@
 			(project "4mix"
 				(path "/b63493d3-5f6d-47e3-845b-87e7090fc1ab/d0b612c1-0c25-4058-bf92-38ae27a09cef"
-					(reference "R58")
+					(reference "R93")
 					(unit 1)
 				)
@@
 		(dnp no)
 		(fields_autoplaced yes)
-		(property "Reference" "R57"
+		(property "Reference" "R92"
 			(at 115.57 57.15 90)
 			(effects
@@
 			(project "4mix"
 				(path "/b63493d3-5f6d-47e3-845b-87e7090fc1ab/d0b612c1-0c25-4058-bf92-38ae27a09cef"
-					(reference "R57")
+					(reference "R92")
 					(unit 1)
 				)
@@
 		(on_board yes)
 		(dnp no)
-		(property "Reference" "#PWR028"
+		(property "Reference" "#PWR038"
 			(at 251.46 102.87 0)
 			(effects
@@
 			(project "4mix"
 				(path "/b63493d3-5f6d-47e3-845b-87e7090fc1ab/d0b612c1-0c25-4058-bf92-38ae27a09cef"
-					(reference "#PWR028")
+					(reference "#PWR038")
 					(unit 1)
 				)
@@
 		(dnp no)
 		(fields_autoplaced yes)
-		(property "Reference" "R55"
+		(property "Reference" "R90"
 			(at 59.69 55.88 90)
 			(effects
@@
 			(project "4mix"
 				(path "/b63493d3-5f6d-47e3-845b-87e7090fc1ab/d0b612c1-0c25-4058-bf92-38ae27a09cef"
-					(reference "R55")
+					(reference "R90")
 					(unit 1)
 				)
@@
 		(on_board yes)
 		(dnp no)
-		(property "Reference" "U8"
+		(property "Reference" "U11"
 			(at 243.332 93.218 90)
 			(effects
@@
 			(project "4mix"
 				(path "/b63493d3-5f6d-47e3-845b-87e7090fc1ab/d0b612c1-0c25-4058-bf92-38ae27a09cef"
-					(reference "U8")
+					(reference "U11")
 					(unit 3)
 				)
@@
 		(dnp no)
 		(fields_autoplaced yes)
-		(property "Reference" "R56"
+		(property "Reference" "R91"
 			(at 77.47 67.31 90)
 			(effects
@@
 			(project "4mix"
 				(path "/b63493d3-5f6d-47e3-845b-87e7090fc1ab/d0b612c1-0c25-4058-bf92-38ae27a09cef"
-					(reference "R56")
-					(unit 1)
-				)
+					(reference "R91")
+					(unit 1)
+				)
