File: modules/4mix/4mix.kicad_sch (KiCad schematic)
At the start: 75 parts, among them U1 MCP6002-xSN, U2 MCP6002-xSN, U3 MCP6002-xSN, U4 MCP6002-xSN, U5 MCP6002-xSN, U6 MCP6002-xSN

Commit message: Add routes for mian mix
Parts:
- removed R9: 100, Resistor_SMD:R_0402_1005Metric, symbol Device:R
Connections:
- net at R11.1: now also C3.1, R5.2, U1.1
Changed lines of the file:
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@@
 		)
 	)
-	(text "This sits close to the summing amp\n"
-		(exclude_from_sim no)
-		(at 113.792 126.492 0)
-		(effects
-			(font
-				(size 1.27 1.27)
-			)
-			(justify left)
-		)
-	)
 	(text "# Sends Mix"
 		(exclude_from_sim no)
@@
 	(wire
 		(pts
-			(xy 99.06 121.92) (xy 111.76 121.92)
-		)
-		(stroke
-			(width 0)
-			(type default)
-		)
-	)
-	(wire
-		(pts
 			(xy 137.16 339.09) (xy 143.51 339.09)
 		)
@@
 	(wire
 		(pts
-			(xy 85.09 121.92) (xy 91.44 121.92)
+			(xy 85.09 121.92) (xy 111.76 121.92)
 		)
 		(stroke
@@
 					(unit 1)
 				)
-			)
-		)
-	)
-	(symbol
-		(lib_id "Device:R")
-		(at 95.25 121.92 90)
-		(unit 1)
-		(exclude_from_sim no)
-		(in_bom yes)
-		(on_board yes)
-		(dnp no)
-		(fields_autoplaced yes)
-		(property "Reference" "R9"
-			(at 95.25 115.57 90)
-			(effects
-				(font
-					(size 1.27 1.27)
-				)
-			)
-		)
-		(property "Value" "100"
-			(at 95.25 118.11 90)
-			(effects
-				(font
-					(size 1.27 1.27)
-				)
-			)
-		)
-		(property "Footprint" "Resistor_SMD:R_0402_1005Metric"
-			(at 95.25 123.698 90)
-			(effects
-				(font
-					(size 1.27 1.27)
-				)
-				(hide yes)
-			)
-		)
-		(property "Datasheet" "~"
-			(at 95.25 121.92 0)
-			(effects
-				(font
-					(size 1.27 1.27)
-				)
-				(hide yes)
-			)
-		)
-		(property "Description" "Resistor"
-			(at 95.25 121.92 0)
-			(effects
-				(font
-					(size 1.27 1.27)
-				)
-				(hide yes)
-			)
-		)
-		(pin "2"
-		)
-		(pin "1"
-		)
-		(instances
-			(project "4mix"
-				(path "/b63493d3-5f6d-47e3-845b-87e7090fc1ab"
-					(reference "R9")
-					(unit 1)
-				)
