File: opt/Breakouts/ESP32S3/esp32-s3.kicad_pcb (KiCad board)
At the start: 2 copper layers, 30.5 x 68.6 mm, 16 parts, among them J5 USB_C_Receptacle_USB2.0_14P, SW1 K2-1808SN-A4SW-01, SW2 K2-1808SN-A4SW-01, U1 ESP32-S3-WROOM-1

Commit message: Finish adding the breakout
Parts:
- added INPUT2: Conn_01x02_Socket, Connector_PinSocket_2.54mm:PinSocket_1x02_P2.54mm_Vertical, B.Cu at (49.3, 77.7)
- INPUT1, OUTPUT1: moved to B.Cu
- U1: value ESP32-S3-WROOM-1 -> ESP32-S3-WROOM-1U-N16R8
- moved C4 69.9 mm to (48.8, 48.5)
- moved R3 69.5 mm to (52.1, 47.8), turned to 90 degrees
- moved C3 69.5 mm to (48.8, 47.2)
- moved C1 57.9 mm to (57.3, 53.3)
- moved R11 56.9 mm to (64.7, 47.8)
- moved C2 54.2 mm to (54.1, 53.3), turned to 180 degrees
- moved C20 48.5 mm to (75.4, 51.1), turned to 180 degrees
- moved R4 46.5 mm to (72.6, 52.1), turned to -90 degrees
- turned INPUT1 to 180 degrees
- turned OUTPUT1 to 180 degrees
Connections:
- net Net-(SW1-B) renamed IO0
- net Net-(SW2-B) renamed EN
Routing:
- net IO0: track 0.00 -> 70.5 mm, vias 0 -> 2
- net EN: track 0.00 -> 50.3 mm
- net USB_D+: track 0.00 -> 39.0 mm, vias 0 -> 2
- net USB_D-: track 0.00 -> 35.3 mm
- net GND: track 10.2 -> 37.8 mm, vias 0 -> 9
- net RX: track 0.00 -> 23.8 mm, vias 0 -> 2
- net Net-(J5-SHIELD): track 0.00 -> 20.7 mm
- net V_SUPPLY: track 10.2 -> 25.9 mm, vias 0 -> 3
- net IO17: track 0.00 -> 8.93 mm
- net Net-(J5-CC2): track 0.00 -> 7.83 mm
- net IO16: track 0.00 -> 7.66 mm
- net Net-(J5-VBUS-PadA4): track 0.00 -> 7.58 mm
- net IO41: track 0.00 -> 6.79 mm
- net IO15: track 0.00 -> 6.19 mm
- net IO7: track 0.00 -> 5.95 mm
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- added copper zone on B.Cu, net GND
Other:
- board text added: "0"
- board text added: "15"
- board text added: "16"
- board text added: "17"
- board text added: "35"
- board text added: "36"
- board text added: "37"
- board text added: "38"
- board text added: "39"
- board text added: "4"
- board text added: "40"
- board text added: "41"
- board text added: "5"
- board text added: "6"
- board text added: "7"
- board text added: "EN"
- board text added: "RX"
- board text added: "TX"
