File: opt/Breakouts/ESP32S3/esp32-s3.kicad_sch (KiCad schematic)
At the start: 20 parts, among them J5 USB_C_Receptacle_USB2.0_14P, SW1 K2-1808SN-A4SW-01, SW2 K2-1808SN-A4SW-01, U1 ESP32-S3-WROOM-1

Commit message: Finish adding the breakout
Parts:
- removed C5: 100uf, Capacitor_SMD:C_1206_3216Metric, symbol Device:C
- removed C6: 0.1uf, Capacitor_SMD:C_0402_1005Metric, symbol Device:C
- added INPUT2: Conn_01x02_Socket, Connector_PinSocket_2.54mm:PinSocket_1x02_P2.54mm_Vertical, symbol Connector:Conn_01x02_Socket
- U1: value ESP32-S3-WROOM-1 -> ESP32-S3-WROOM-1U-N16R8
Connections:
- net EN: now reaches C3.2, C4.2, R3.2, SW2.2 (B), U1.3 (EN)
- net EN: now also INPUT2.1 (Pin_1)
- net IO0: now reaches SW1.2 (B), U1.27 (IO0)
- net IO0: now also INPUT2.2 (Pin_2)
