File: modules/imix/imix.kicad_sch (KiCad schematic)
At the start: 39 parts, among them U1 MCP6002-xSN, U2 MCP6002-xSN, U3 MCP6002-xSN

Commit message: Add improved schematics
Parts:
- added C1, C13, C2, C3, C4: 100pf, Capacitor_SMD:C_0402_1005Metric, symbol Device:C
- added C10, C11, C12, C15, C7: 0.1uf, Capacitor_SMD:C_0402_1005Metric, symbol Device:C
- added C5, C6, C8, C9: 10uf, Capacitor_SMD:C_0402_1005Metric, symbol Device:C
- added R13, R14, R15, R16, R21, R22, R23, R24: 100, Resistor_SMD:R_0402_1005Metric, symbol Device:R
- added R29: 10, Resistor_SMD:R_0402_1005Metric, symbol Device:R
- R10: renamed from R19; value 100k -> 22k
- R11: renamed from R13; value 100k -> 22k
- R12: renamed from R15; value 100k -> 22k
- R17: renamed from R4; value 200k -> 22k
- R18: renamed from R6; value 200k -> 22k
- R19: renamed from R8; value 200k -> 22k
- R20: renamed from R10; value 200k -> 22k
- R25: renamed from R11; value 200k -> 22k
- R27: renamed from R1; value 1k -> 10k
- R28: renamed from R2; value 1k -> 10k
- R5: renamed from R20; value 100k -> 22k
- R6: renamed from R18; value 100k -> 22k
- R7: renamed from R16; value 100k -> 22k
- R8: renamed from R14; value 100k -> 22k
- R9: renamed from R17; value 100k -> 22k
- renumbered C2 to C14, C3 to C16, C1 to C17, C4 to C18, R3 to R1, R5 to R2, R12 to R26, R9 to R3, R7 to R4, RV3 to RV1, RV4 to RV2, RV1 to RV3, RV2 to RV4, U2 to U1, U1 to U2
Connections:
- net GND: now also C16.2, C10.2, C11.2, C12.2, C15.2, C5.2, C6.2, C7.2, C8.2, C9.2
- net V_MID: now also R21.2, R22.2, R23.2, R24.2, R29.2; no longer C16.2, R1.1, R2.1, R27.2, R28.1, R3.1, R4.1, RV1.1, RV2.1, RV3.1, RV4.1, U1.3 (+), U1.5 (+), U2.3 (+), U2.5 (+)
- net V_SUPPLY: no longer C16.1
- net at R9.2, U1.1: now also C1.2, R13.1; no longer RV1.3
- net at R10.1, R5.2, U1.6 (-): now also C2.1
- net at R10.2, U1.7: now also C2.2, R14.1; no longer RV2.3
- net at R17.2, R18.2, R19.2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: now also C13.1
- net at R25.2, R26.1, U3.1: now also C13.2
- net at R12.1, R7.2, U2.6 (-): now also C4.1
- net at U3.5 (+): now also C16.1, R27.2, R28.1, C15.1
- net at U3.6 (-): now also U3.7, R29.1
- net at R11.2, U2.1: now also C3.2, R15.1; no longer RV3.3
- net at R12.2, U2.7: now also C4.2, R16.1; no longer RV4.3
- net at R6.2, R9.1, U1.2 (-): now also C1.1
- net at R11.1, R8.2, U2.2 (-): now also C3.1
- new net: R14.2, RV2.3
- new net: R13.2, RV1.3
- new net: R16.2, RV4.3
- new net: R15.2, RV3.3
- new net V_MID_1: C5.1, C7.1, R21.1, R4.1, RV3.1, U2.3 (+)
- new net V_MID_2: C10.1, C6.1, R22.1, R3.1, RV4.1, U2.5 (+)
- new net V_MID_3: C12.1, C9.1, R1.1, R24.1, RV1.1, U1.3 (+)
- new net V_MID_4: C11.1, C8.1, R2.1, R23.1, RV2.1, U1.5 (+)
Other:
- moved on the sheet: C14, C16, C17, C18, R11, R19, R25, R26, R27, R28, R4, R8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

Commit message: Start placing the PCB
Parts:
- renumbered RV3 to RV1, RV4 to RV2, RV1 to RV3, RV2 to RV4
Changed lines of the file:
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@@
 		(on_board yes)
 		(dnp no)
-		(property "Reference" "RV1"
+		(property "Reference" "RV3"
 			(at 104.14 156.972 90)
 			(effects
@@
 			(project "i_mix"
 				(path "/b63493d3-5f6d-47e3-845b-87e7090fc1ab"
-					(reference "RV1")
+					(reference "RV3")
 					(unit 1)
 				)
@@
 		(on_board yes)
 		(dnp no)
-		(property "Reference" "RV2"
+		(property "Reference" "RV4"
 			(at 104.14 203.962 90)
 			(effects
@@
 			(project "i_mix"
 				(path "/b63493d3-5f6d-47e3-845b-87e7090fc1ab"
-					(reference "RV2")
+					(reference "RV4")
 					(unit 1)
 				)
@@
 		(on_board yes)
 		(dnp no)
-		(property "Reference" "RV3"
+		(property "Reference" "RV1"
 			(at 107.95 45.212 90)
 			(effects
@@
 			(project ""
 				(path "/b63493d3-5f6d-47e3-845b-87e7090fc1ab"
-					(reference "RV3")
+					(reference "RV1")
 					(unit 1)
 				)
@@
 		(on_board yes)
 		(dnp no)
-		(property "Reference" "RV4"
+		(property "Reference" "RV2"
 			(at 107.95 99.822 90)
 			(effects
@@
 			(project "i_mix"
 				(path "/b63493d3-5f6d-47e3-845b-87e7090fc1ab"
-					(reference "RV4")
+					(reference "RV2")
 					(unit 1)
 				)
