File: modules/32bit-5v/32bit-5v.kicad_sch (KiCad schematic)
At the start: 61 parts, among them J5 USB_C_Receptacle_USB2.0_14P, SW1 K2-1808SN-A4SW-01, SW2 K2-1808SN-A4SW-01, SW4 K2-1808SN-A4SW-01, U1 ESP32-S3-WROOM-1U-N16R8, U3 MCP6002-xSN, U4 ES8388, U5 AP2112K-3.3

Commit message: Checkpoint 32bit-5V Basic Economy passive bindings and matched HOLD production evidence
Parts:
- C1, C21, C22, C26, C34, C36, C39, C4, C6: Dielectric (none) -> X7R; ESR (none) -> UNVERIFIED at application frequency/temperature; Effective Capacitance (none) -> UNVERIFIED at operating DC bias/temperature; not nominal ca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; LCSC (none) -> C1525; MPN (none) -> CL05B104KO5NNNC; Manufacturer (none) -> Samsung Electro-Mechanics; Polarity (none) -> Nonpolar; Sourcing Review (none) -> HOLD - exact Basic catalog binding; application/rating sign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; Temperature Rating (none) -> -55 to +125 C; Tolerance (none) -> ±10%; Voltage Rating (none) -> 16V
- C2, C8: Dielectric (none) -> X5R; ESR (none) -> UNVERIFIED at application frequency/temperature; Effective Capacitance (none) -> UNVERIFIED at operating DC bias/temperature; not nominal ca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; LCSC (none) -> C19702; MPN (none) -> CL10A106KP8NNNC; Manufacturer (none) -> Samsung Electro-Mechanics; Polarity (none) -> Nonpolar; Sourcing Review (none) -> HOLD - exact Basic catalog binding; application/rating sign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; Temperature Rating (none) -> -55 to +85 C; Tolerance (none) -> ±10%; Voltage Rating (none) -> 10V
- C20: Dielectric (none) -> X7R; ESR (none) -> UNVERIFIED at application frequency/temperature; Effective Capacitance (none) -> UNVERIFIED at operating DC bias/temperature; not nominal ca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; LCSC (none) -> C1710; MPN (none) -> CL21B103KBANNNC; Manufacturer (none) -> Samsung Electro-Mechanics; Polarity (none) -> Nonpolar; Sourcing Review (none) -> HOLD - exact Basic catalog binding; application/rating sign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; Temperature Rating (none) -> -55 to +125 C; Tolerance (none) -> ±10%; Voltage Rating (none) -> 50V
- C27, C33, C35, C37, C38, C5: Dielectric (none) -> X5R; ESR (none) -> UNVERIFIED at application frequency/temperature; Effective Capacitance (none) -> UNVERIFIED at operating DC bias/temperature; not nominal ca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; LCSC (none) -> C15525; MPN (none) -> CL05A106MQ5NUNC; Manufacturer (none) -> Samsung Electro-Mechanics; Polarity (none) -> Nonpolar; Sourcing Review (none) -> HOLD - exact Basic catalog binding; application/rating sign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; Temperature Rating (none) -> -55 to +85 C; Tolerance (none) -> ±20%; Voltage Rating (none) -> 6.3V
- C3: Dielectric (none) -> X5R; ESR (none) -> UNVERIFIED at application frequency/temperature; Effective Capacitance (none) -> UNVERIFIED at operating DC bias/temperature; not nominal ca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; LCSC (none) -> C52923; MPN (none) -> CL05A105KA5NQNC; Manufacturer (none) -> Samsung Electro-Mechanics; Polarity (none) -> Nonpolar; Sourcing Review (none) -> HOLD - exact Basic catalog binding; application/rating sign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; Temperature Rating (none) -> -55 to +85 C; Tolerance (none) -> ±10%; Voltage Rating (none) -> 25V
- C40: Dielectric (none) -> X5R; ESR (none) -> UNVERIFIED at application frequency/temperature; Effective Capacitance (none) -> UNVERIFIED at operating DC bias/temperature; not nominal ca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; Polarity (none) -> Nonpolar; Sourcing Review (none) -> HOLD - exact Basic catalog binding; application/rating sign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; Temperature Rating (none) -> -55 to +85 C; Tolerance (none) -> ±10%; Voltage Rating (none) -> 25V
- C41: Dielectric (none) -> X5R; ESR (none) -> UNVERIFIED at application frequency/temperature; Effective Capacitance (none) -> UNVERIFIED at operating DC bias/temperature; not nominal ca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; Polarity (none) -> Nonpolar; Sourcing Review (none) -> HOLD - exact Basic catalog binding; application/rating sign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; Temperature Rating (none) -> -55 to +85 C; Tolerance (none) -> ±20%; Voltage Rating (none) -> 25V
- C42: Dielectric (none) -> X7R; ESR (none) -> UNVERIFIED at application frequency/temperature; Effective Capacitance (none) -> UNVERIFIED at operating DC bias/temperature; not nominal ca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; Manufacturer Samsung -> Samsung Electro-Mechanics; Polarity (none) -> Nonpolar; Sourcing Review (none) -> HOLD - exact Basic catalog binding; application/rating sign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; Temperature Rating (none) -> -55 to +125 C; Tolerance (none) -> ±10%; Voltage Rating (none) -> 16V
- C7: Dielectric (none) -> X5R; ESR (none) -> UNVERIFIED at application frequency/temperature; Effective Capacitance (none) -> UNVERIFIED at operating DC bias/temperature; not nominal ca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; LCSC (none) -> C15008; MPN (none) -> CL31A107MQHNNNE; Manufacturer (none) -> Samsung Electro-Mechanics; Polarity (none) -> Nonpolar; Sourcing Review (none) -> HOLD - exact Basic catalog binding; application/rating sign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; Temperature Rating (none) -> -55 to +85 C; Tolerance (none) -> ±20%; Voltage Rating (none) -> 6.3V
- FB1: LCSC (none) -> C5671; MPN (none) -> GZ2012D121TF; Manufacturer (none) -> Sunlord
- J5: LCSC (none) -> C165948; MPN (none) -> TYPE-C-31-M-12; Manufacturer (none) -> Korean Hroparts Elec
- R1, R13, R17, R2, R9: LCSC (none) -> C11702; MPN (none) -> 0402WGF1001TCE; Manufacturer (none) -> UNI-ROYAL(Uniroyal Elec); Power Derating (none) -> 50% continuous at <=70 C; intended rail/signal envelope only; Power Rating (none) -> 0.0625W at <=70 C; derate above 70 C; Sourcing Review (none) -> HOLD - exact Basic catalog binding; application/rating sign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; Temperature Rating (none) -> -55 to +155 C; Tolerance (none) -> ±1%; Voltage Rating (none) -> 50V
- R10, R12, R16, R19: LCSC (none) -> C25741; MPN (none) -> 0402WGF1003TCE; Manufacturer (none) -> UNI-ROYAL(Uniroyal Elec); Power Derating (none) -> 50% continuous at <=70 C; intended rail/signal envelope only; Power Rating (none) -> 0.0625W at <=70 C; derate above 70 C; Sourcing Review (none) -> HOLD - exact Basic catalog binding; application/rating sign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; Temperature Rating (none) -> -55 to +155 C; Tolerance (none) -> ±1%; Voltage Rating (none) -> 50V
- R11, R4: LCSC (none) -> C23186; MPN (none) -> 0603WAF5101T5E; Manufacturer (none) -> UNI-ROYAL(Uniroyal Elec); Power Derating (none) -> 50% continuous at <=70 C; intended rail/signal envelope only; Power Rating (none) -> 0.1W at <=70 C; derate above 70 C; Sourcing Review (none) -> HOLD - exact Basic catalog binding; application/rating sign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; Temperature Rating (none) -> -55 to +155 C; Tolerance (none) -> ±1%; Voltage Rating (none) -> 75V
- R14, R18, R26, R7, R8: LCSC (none) -> C25105; MPN (none) -> 0402WGF330JTCE; Manufacturer (none) -> UNI-ROYAL(Uniroyal Elec); Power Derating (none) -> 50% continuous at <=70 C; pulse/load qualification HOLD; Power Rating (none) -> 0.0625W at <=70 C; derate above 70 C; Sourcing Review (none) -> HOLD - exact Basic catalog binding; application/rating sign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; Temperature Rating (none) -> -55 to +155 C; Tolerance (none) -> ±1%; Voltage Rating (none) -> 50V
- R15: LCSC (none) -> C22859; MPN (none) -> 0603WAF100JT5E; Manufacturer (none) -> UNI-ROYAL(Uniroyal Elec); Power Derating (none) -> 50% continuous at <=70 C; pulse/load qualification HOLD; Power Rating (none) -> 0.1W at <=70 C; derate above 70 C; Sourcing Review (none) -> HOLD - exact Basic catalog binding; application/rating sign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; Temperature Rating (none) -> -55 to +155 C; Tolerance (none) -> ±1%; Voltage Rating (none) -> 75V
- R24, R25: LCSC (none) -> C25900; MPN (none) -> 0402WGF4701TCE; Manufacturer (none) -> UNI-ROYAL(Uniroyal Elec); Power Derating (none) -> 50% continuous at <=70 C; intended rail/signal envelope only; Power Rating (none) -> 0.0625W at <=70 C; derate above 70 C; Sourcing Review (none) -> HOLD - exact Basic catalog binding; application/rating sign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; Temperature Rating (none) -> -55 to +155 C; Tolerance (none) -> ±1%; Voltage Rating (none) -> 50V
- R3: LCSC (none) -> C25744; MPN (none) -> 0402WGF1002TCE; Manufacturer (none) -> UNI-ROYAL(Uniroyal Elec); Power Derating (none) -> 50% continuous at <=70 C; intended rail/signal envelope only; Power Rating (none) -> 0.0625W at <=70 C; derate above 70 C; Sourcing Review (none) -> HOLD - exact Basic catalog binding; application/rating sign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; Temperature Rating (none) -> -55 to +155 C; Tolerance (none) -> ±1%; Voltage Rating (none) -> 50V
- R5, R6: LCSC (none) -> C25867; MPN (none) -> 0402WGF1501TCE; Manufacturer (none) -> UNI-ROYAL(Uniroyal Elec); Power Derating (none) -> 50% continuous at <=70 C; intended rail/signal envelope only; Power Rating (none) -> 0.0625W at <=70 C; derate above 70 C; Sourcing Review (none) -> HOLD - exact Basic catalog binding; application/rating sign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; Temperature Rating (none) -> -55 to +155 C; Tolerance (none) -> ±1%; Voltage Rating (none) -> 50V
- SW1, SW2, SW4: LCSC (none) -> C92589; MPN (none) -> K2-1808SN-A4SW-01; Manufacturer (none) -> Korean Hroparts Elec
- U1: LCSC (none) -> C3013946; MPN (none) -> ESP32-S3-WROOM-1U-N16R8; Manufacturer (none) -> Espressif Systems; Sourcing Review (none) -> HOLD - C3013946 Standard-only componentProductType=2; exact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
- U3: LCSC (none) -> C116706; MPN (none) -> MCP6002-I/SN; Manufacturer (none) -> Microchip Tech
- U4: LCSC (none) -> C365736
