File: modules/32bit-5v/32bit-5v.kicad_pcb (KiCad board)
At the start: 4 copper layers, 30.5 x 68.6 mm, 65 parts, among them J5 USB_C_Receptacle_USB2.0_14P, SW1 K2-1808SN-A4SW-01, SW2 K2-1808SN-A4SW-01, SW4 K2-1808SN-A4SW-01, U1 ESP32-S3-WROOM-1U-N16R8, U3 MCP6002-xSN, U5 AP7361C-33E-13

Commit message: Finish 32-bit 5V multilayer routing and exports; retain approved THT placement
Parts:
- removed C10, C11, C12, C13, C9: 100uf, Capacitor_SMD:C_1206_3216Metric
- added C42: 0.1uf, Capacitor_SMD:C_0402_1005Metric, F.Cu at (56.8, 49.0)
- C40, C41: moved to F.Cu
- J5: footprint BreadModular_TypeC:HRO-TYPE-C-31-M-12 -> Module32:HRO-TYPE-C-31-M-12
- U3: footprint Package_SO:SOIC-8-1EP_3.9x4.9mm_P1.27mm_EP2.29x3mm -> Package_SO:SOIC-8_3.9x4.9mm_P1.27mm
- U4: value ~ -> ES8388; footprint Package_DFN_QFN:QFN-28-1EP_4x4mm_P0.45mm_EP2.4x2.4mm_ThermalVias -> Module32:ES8388_QFN28_4x4_P0.45_EP2.6_ThermalVias
- U5: value AP7361C-33E-13 -> AP2112K-3.3; footprint Package_TO_SOT_SMD:SOT-223-3_TabPin2 -> Package_TO_SOT_SMD:SOT-23-5; moved to F.Cu
- moved C40 14.9 mm to (55.3, 47.0), turned to 0 degrees
- moved U5 10.1 mm to (60.5, 47.5), turned to 0 degrees
- moved C41 7.99 mm to (65.0, 53.0), turned to 0 degrees
Connections:
- U5 pad 3: +3V3 -> +5V
Routing:
- net +3V3_ESP32: track 62.8 -> 39.5 mm, vias 7 -> 3
- net GND: track 76.1 -> 69.0 mm, vias 36 -> 31
- net +5V: track 17.4 -> 23.5 mm
- net +3V3: track 110.9 -> 114.1 mm, vias 6 -> 7

Commit message: Update the 32bit-5v production files.
Other:
- board text added: "32BIT 2.0.0"
- board text removed: "32BIT 0.3.0"
