File: modules/16bit-5v/16bit-5v.kicad_pcb (KiCad board)
At the start: 2 copper layers, 30.5 x 68.6 mm, 62 parts, among them J1 Conn_01x08_Socket, J2 Conn_01x08_Socket, J5 USB_C_Receptacle_USB2.0_14P, SW1 K2-1808SN-A4SW-01, SW2 K2-1808SN-A4SW-01, SW3 K2-1808SN-A4SW-01, U1 RP2350_60QFN, U2 W25Q128JVS, U3 MCP6002-xSN, U4 PT8211, U5 PSRAM, U6 AP2112K-3.3, Y1 ABM8-272-T3

Commit message: Integrate verified 16bit-5v exports and THT placement approval
Parts:
- J1, J2: value Conn_01x08_Socket -> Conn_01x05_Socket
- U3: footprint Package_SO:SOIC-8-1EP_3.9x4.9mm_P1.27mm_EP2.29x3mm -> Package_SO:SOIC-8_3.9x4.9mm_P1.27mm
- U4: value PT8211 -> PT8211-S; footprint Package_SO:SOIC-8-1EP_3.9x4.9mm_P1.27mm_EP2.29x3mm -> Package_SO:SOIC-8_3.9x4.9mm_P1.27mm
- moved C12 5.62 mm to (69.2, 59.3), turned to 0 degrees
- moved L1 5.47 mm to (67.8, 64.6), turned to -90 degrees
- moved C7 2.16 mm to (68.3, 62.3)
- moved R5 1.91 mm to (69.9, 63.7), turned to 0 degrees
- moved C9 1.11 mm to (72.0, 66.3)
- moved C6 1.02 mm to (69.9, 66.1)
- moved C26 0.38 mm to (74.0, 50.1)
Connections:
- net Net-(J5-VBUS-PadA4) renamed /USB_VBUS_UNUSED
- J5 pad A8: (no net) -> unconnected-(J5-SBU1-PadA8)
- J5 pad B8: (no net) -> unconnected-(J5-SBU2-PadB8)
Routing:
- net +3V3: track 37.5 -> 52.8 mm, vias 15 -> 19
- net /VREG_LX: track 10.0 -> 1.90 mm
- net /USB_VBUS_UNUSED: track 0.00 -> 7.30 mm, vias 0 -> 2
- net +1V1: track 21.8 -> 14.6 mm
- net GND: track 88.1 -> 93.7 mm, vias 35 -> 37
- net /VREG_AVDD: track 7.39 -> 10.9 mm

Commit message: Checkpoint 16bit-5V Basic/Economy passive sourcing with explicit electrical and assembly holds
Parts:
- C1, C5: value 0.1uf -> 0.1uF
- C20, C22, C23: value 10nf -> 10nF
- C21: value 100uf -> 100uF

Commit message: Add 16bit 5v as 2.0.0
Parts:
- D1: value LED -> KT-0603R
- U4: value PT8211-S -> TM8211-TA2302
- U5: value PSRAM -> APS6404L-3SQR-SN
- moved C27 5.47 mm to (71.2, 55.0), turned to 180 degrees
Routing:
- net GND: track 93.7 -> 97.5 mm, vias 37 -> 39
- net +3V3: track 52.8 -> 50.9 mm, vias 19 -> 17
Other:
- board text added: "16BIT 2.0.0"
- board text removed: "16BIT 1.0.0"
