File: modules/16bit-5v/16bit-5v.kicad_sch (KiCad schematic)
At the start: 63 parts, among them J1 Conn_01x08_Socket, J2 Conn_01x08_Socket, J5 USB_C_Receptacle_USB2.0_14P, SW1 K2-1808SN-A4SW-01, SW2 K2-1808SN-A4SW-01, SW3 K2-1808SN-A4SW-01, U1 RP2350_60QFN, U2 W25Q128JVS, U3 MCP6002-xSN, U4 PT8211, U5 PSRAM, U6 AP2112K-3.3, Y1 ABM8-272-T3

Commit message: Integrate verified 16bit-5v exports and THT placement approval
Parts:
- J1, J2: value Conn_01x08_Socket -> Conn_01x05_Socket
- J5: symbol Connector:USB_C_Receptacle_USB2.0_14P -> Bread16bit:USB_C_HRO_TYPE_C_31_M_12; JLCPCB Position Offset X (none) -> 0; JLCPCB Position Offset Y (none) -> -3.675
- U3: footprint Package_SO:SOIC-8-1EP_3.9x4.9mm_P1.27mm_EP2.29x3mm -> Package_SO:SOIC-8_3.9x4.9mm_P1.27mm
- U4: value PT8211 -> PT8211-S; footprint Package_SO:SOIC-8-1EP_3.9x4.9mm_P1.27mm_EP2.29x3mm -> Package_SO:SOIC-8_3.9x4.9mm_P1.27mm; symbol Audio:PT8211 -> Bread16bit:PT8211
Connections:
- net GND: no longer J5.B1 (GND), J5.B12 (GND)
- net USB_VBUS_UNUSED: now reaches J5.A4 (VBUS), J5.A9 (VBUS)
- net USB_VBUS_UNUSED: no longer J5.B4 (VBUS), J5.B9 (VBUS)
- no-connect marks 0 -> 18
Changed lines of the file:
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@@
 			)
 		)
-		(property "Value" "Conn_01x08_Socket"
+		(property "Value" "Conn_01x05_Socket"
 			(at 455.93 121.158 90)
 			(effects
@@
 	)
 	(symbol
-		(lib_id "Audio:PT8211")
+		(lib_id "Bread16bit:PT8211")
 		(at 262.89 317.5 0)
 		(unit 1)
@@
 			)
 		)
-		(property "Value" "PT8211"
+		(property "Value" "PT8211-S"
 			(at 248.666 320.294 0)
 			(effects
@@
 			)
 		)
-		(property "Footprint" "Package_SO:SOIC-8-1EP_3.9x4.9mm_P1.27mm_EP2.29x3mm"
+		(property "Footprint" "Package_SO:SOIC-8_3.9x4.9mm_P1.27mm"
 			(at 262.89 332.74 0)
 			(effects
@@
 			)
 		)
-		(property "Footprint" "Package_SO:SOIC-8-1EP_3.9x4.9mm_P1.27mm_EP2.29x3mm"
+		(property "Footprint" "Package_SO:SOIC-8_3.9x4.9mm_P1.27mm"
 			(at 66.04 321.31 0)
 			(effects
@@
 	)
 	(symbol
-		(lib_id "Connector:USB_C_Receptacle_USB2.0_14P")
+		(lib_id "Bread16bit:USB_C_HRO_TYPE_C_31_M_12")
 		(at 40.64 46.99 0)
 		(unit 1)
@@
 			)
 		)
-		(property "Description" "USB 2.0-only 14P Type-C Receptacle connector"
+		(property "Description" "HRO TYPE-C-31-M-12: 12 solder terminals; A1/B12, A12/B1, A4/B9, A9/B4 share lands; A8/B8 are unused SBU"
 			(at 40.64 46.99 0)
 			(effects
@@
 		(pin "B7"
 		)
-		(pin "B9"
-		)
 		(pin "B5"
 		)
@@
 		(pin "A6"
 		)
-		(pin "B12"
-		)
-		(pin "B4"
-		)
 		(pin "A1"
 		)
@@
 		(pin "A9"
 		)
-		(pin "B1"
-		)
 		(pin "S1"
 		)
@@
 		(pin "A4"
 		)
-		(instances
+		(property "JLCPCB Position Offset X" "0" (at 40.64 46.99 0) (effects (font (size 1.27 1.27)) (hide yes)))
+(property "JLCPCB Position Offset Y" "-3.675" (at 40.64 46.99 0) (effects (font (size 1.27 1.27)) (hide yes)))
+(instances
 			(project "RP2350_60QFN_minimal"
 				(path "/94683f5c-9cd9-448e-be96-9792537b5cb8"
@@
 			)
 		)
-	)
+(pin "A8")
+(pin "B8"))
 	(symbol
 		(lib_id "power:GND")
@@
 			)
 		)
-		(property "Footprint" "Package_SO:SOIC-8-1EP_3.9x4.9mm_P1.27mm_EP2.29x3mm"
+		(property "Footprint" "Package_SO:SOIC-8_3.9x4.9mm_P1.27mm"
 			(at 532.13 201.93 0)
 			(effects
@@
 			)
 		)
-		(property "Footprint" "Package_SO:SOIC-8-1EP_3.9x4.9mm_P1.27mm_EP2.29x3mm"
+		(property "Footprint" "Package_SO:SOIC-8_3.9x4.9mm_P1.27mm"
 			(at 66.04 370.84 0)
 			(effects
@@
 			)
 		)
-		(property "Value" "Conn_01x08_Socket"
+		(property "Value" "Conn_01x05_Socket"
 			(at 516.382 120.142 90)
 			(effects
@@
 		)
 	)
+(no_connect (at 166.37 176.53))
+(no_connect (at 166.37 179.07))
+(no_connect (at 229.87 127.0))
+(no_connect (at 229.87 129.54))
+(no_connect (at 229.87 132.08))
+(no_connect (at 229.87 134.62))
+(no_connect (at 229.87 137.16))
+(no_connect (at 229.87 139.7))
+(no_connect (at 229.87 147.32))
+(no_connect (at 229.87 149.86))
+(no_connect (at 229.87 152.4))
+(no_connect (at 229.87 154.94))
+(no_connect (at 229.87 157.48))
+(no_connect (at 229.87 165.1))
+(no_connect (at 229.87 167.64))
+(no_connect (at 229.87 170.18))
+(no_connect (at 229.87 172.72))
+(no_connect (at 229.87 175.26))
+(symbol
+		(lib_id "power:PWR_FLAG")
+		(at 267.9700 144.7800 0)
+		(unit 1)
+		(exclude_from_sim no)
+		(in_bom yes)
+		(on_board yes)
+		(dnp no)
+		(property "Reference" "#FLG0301"
+			(at 267.9700 146.6850 0)
+			(effects
+				(font
+					(size 1.27 1.27)
+				)
+				(hide yes)
+			)
+		)
+		(property "Value" "PWR_FLAG"
+			(at 267.9700 140.9700 0)
+			(effects
+				(font
+					(size 1.27 1.27)
+				)
+			)
+		)
+		(property "Footprint" ""
+			(at 267.9700 144.7800 0)
+			(effects
+				(font
+					(size 1.27 1.27)
+				)
+				(hide yes)
+			)
+		)
+		(property "Datasheet" ""
+			(at 267.9700 144.7800 0)
+			(effects
+				(font
+					(size 1.27 1.27)
+				)
+				(hide yes)
+			)
+		)
+		(property "Description" "Special symbol for telling ERC where power comes from"
+			(at 267.9700 144.7800 0)
+			(effects
+				(font
+					(size 1.27 1.27)
+				)
+				(hide yes)
+			)
+		)
+		(pin "1"
+		)
+		(instances
+			(project "RP2350_60QFN_minimal"
+				(path "/94683f5c-9cd9-448e-be96-9792537b5cb8"
+					(reference "#FLG0301")
+					(unit 1)
+				)
+			)
+		)
+	)
+(symbol
+		(lib_id "power:PWR_FLAG")
+		(at 119.3800 101.6000 0)
+		(unit 1)
+		(exclude_from_sim no)
+		(in_bom yes)
+		(on_board yes)
+		(dnp no)
+		(property "Reference" "#FLG0302"
+			(at 119.3800 103.5050 0)
+			(effects
+				(font
+					(size 1.27 1.27)
+				)
+				(hide yes)
+			)
+		)
+		(property "Value" "PWR_FLAG"
+			(at 119.3800 97.7900 0)
+			(effects
+				(font
+					(size 1.27 1.27)
+				)
+			)
+		)
+		(property "Footprint" ""
+			(at 119.3800 101.6000 0)
+			(effects
+				(font
+					(size 1.27 1.27)
+				)
+				(hide yes)
+			)
+		)
+		(property "Datasheet" ""
+			(at 119.3800 101.6000 0)
+			(effects
+				(font
+					(size 1.27 1.27)
+				)
+				(hide yes)
+			)
+		)
+		(property "Description" "Special symbol for telling ERC where power comes from"
+			(at 119.3800 101.6000 0)
+			(effects
+				(font
+					(size 1.27 1.27)
+				)
+				(hide yes)
+			)
+		)
+		(pin "1"
+		)
+		(instances
+			(project "RP2350_60QFN_minimal"
+				(path "/94683f5c-9cd9-448e-be96-9792537b5cb8"
+					(reference "#FLG0302")
+					(unit 1)
+				)
+			)
+		)
+	)
+(symbol
+		(lib_id "power:PWR_FLAG")
+		(at 166.3700 105.4100 0)
+		(unit 1)
+		(exclude_from_sim no)
+		(in_bom yes)
+		(on_board yes)
+		(dnp no)
+		(property "Reference" "#FLG0303"
+			(at 166.3700 107.3150 0)
+			(effects
+				(font
+					(size 1.27 1.27)
+				)
+				(hide yes)
+			)
+		)
+		(property "Value" "PWR_FLAG"
+			(at 166.3700 101.6000 0)
+			(effects
+				(font
+					(size 1.27 1.27)
+				)
+			)
+		)
+		(property "Footprint" ""
+			(at 166.3700 105.4100 0)
+			(effects
+				(font
+					(size 1.27 1.27)
+				)
+				(hide yes)
+			)
+		)
+		(property "Datasheet" ""
+			(at 166.3700 105.4100 0)
+			(effects
+				(font
+					(size 1.27 1.27)
+				)
+				(hide yes)
+			)
+		)
+		(property "Description" "Special symbol for telling ERC where power comes from"
+			(at 166.3700 105.4100 0)
+			(effects
+				(font
+					(size 1.27 1.27)
+				)
+				(hide yes)
+			)
+		)
+		(pin "1"
+		)
+		(instances
+			(project "RP2350_60QFN_minimal"
+				(path "/94683f5c-9cd9-448e-be96-9792537b5cb8"
+					(reference "#FLG0303")
+					(unit 1)
+				)
+			)
+		)
+	)
+(label "USB_VBUS_UNUSED" (at 55.88 31.75 0) (effects (font (size 1.27 1.27)) (justify left bottom)))
 )

Commit message: Checkpoint 16bit-5V Basic/Economy passive sourcing with explicit electrical and assembly holds
Parts:
- C1, C5: value 0.1uf -> 0.1uF; Dielectric (none) -> X7R; LCSC (none) -> C1525; MPN (none) -> CL05B104KO5NNNC; Manufacturer (none) -> Samsung Electro-Mechanics; Polarity (none) -> nonpolar; Tolerance (none) -> ±10%; Voltage Rating (none) -> 16 V
- C10, C6, C7, C9: Dielectric (none) -> X5R; JLCPCB Application Status (none) -> HOLD: exact supplier review candidate only; effective-C, ES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; LCSC (none) -> C23733; MPN (none) -> CL05A475MP5NRNC; Manufacturer (none) -> Samsung Electro-Mechanics; Polarity (none) -> nonpolar; Tolerance (none) -> ±20%; Voltage Rating (none) -> 10 V
- C11, C12, C13, C14, C15, C16, C17, C18, C2, C24, C8: Dielectric (none) -> X7R; LCSC (none) -> C1525; MPN (none) -> CL05B104KO5NNNC; Manufacturer (none) -> Samsung Electro-Mechanics; Polarity (none) -> nonpolar; Tolerance (none) -> ±10%; Voltage Rating (none) -> 16 V
- C19: Dielectric (none) -> X5R; LCSC (none) -> C15850; MPN (none) -> CL21A106KAYNNNE; Manufacturer (none) -> Samsung Electro-Mechanics; Polarity (none) -> nonpolar; Tolerance (none) -> ±10%; Voltage Rating (none) -> 25 V
- C20: value 10nf -> 10nF; Dielectric (none) -> X7R; LCSC (none) -> C1710; MPN (none) -> CL21B103KBANNNC; Manufacturer (none) -> Samsung Electro-Mechanics; Polarity (none) -> nonpolar; Tolerance (none) -> ±10%; Voltage Rating (none) -> 50 V
- C21: value 100uf -> 100uF; Dielectric (none) -> X5R; JLCPCB Application Status (none) -> HOLD: exact supplier review candidate only; effective-C, ES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; LCSC (none) -> C15008; MPN (none) -> CL31A107MQHNNNE; Manufacturer (none) -> Samsung Electro-Mechanics; Polarity (none) -> nonpolar; Tolerance (none) -> ±20%; Voltage Rating (none) -> 6.3 V
- C22, C23: value 10nf -> 10nF; Dielectric (none) -> X7R; LCSC (none) -> C15195; MPN (none) -> CL05B103KB5NNNC; Manufacturer (none) -> Samsung Electro-Mechanics; Polarity (none) -> nonpolar; Tolerance (none) -> ±10%; Voltage Rating (none) -> 50 V
- C25: Dielectric (none) -> X5R; Manufacturer Samsung -> Samsung Electro-Mechanics; Polarity (none) -> nonpolar; Tolerance (none) -> ±10%; Voltage Rating (none) -> 25 V
- C26: Dielectric (none) -> X7R; Manufacturer Samsung -> Samsung Electro-Mechanics; Polarity (none) -> nonpolar; Tolerance (none) -> ±10%; Voltage Rating (none) -> 16 V
- C27: Dielectric (none) -> X7R; Manufacturer Samsung -> Samsung Electro-Mechanics; Polarity (none) -> nonpolar; Tolerance (none) -> ±10%; Voltage Rating (none) -> 50 V
- C3, C4: Dielectric (none) -> C0G; LCSC (none) -> C1548; MPN (none) -> 0402CG150J500NT; Manufacturer (none) -> FH (Guangdong Fenghua Advanced Tech); Polarity (none) -> nonpolar; Tolerance (none) -> ±5%; Voltage Rating (none) -> 50 V
- J5: LCSC (none) -> C165948; MPN (none) -> TYPE-C-31-M-12; Manufacturer (none) -> Korean Hroparts Elec
- L1: LCSC (none) -> C42411119; MPN (none) -> AOTA-B201610S3R3-101-T; Manufacturer (none) -> Abracon LLC
- R10, R12, R15, R16: LCSC (none) -> C25741; MPN (none) -> 0402WGF1003TCE; Manufacturer (none) -> UNI-ROYAL(Uniroyal Elec); Power Rating (none) -> 62.5 mW; Tolerance (none) -> ±1%; Voltage Rating (none) -> 50 V
- R11, R3: LCSC (none) -> C23186; MPN (none) -> 0603WAF5101T5E; Manufacturer (none) -> UNI-ROYAL(Uniroyal Elec); Power Rating (none) -> 100 mW; Tolerance (none) -> ±1%; Voltage Rating (none) -> 75 V
- R14: LCSC (none) -> C25744; MPN (none) -> 0402WGF1002TCE; Manufacturer (none) -> UNI-ROYAL(Uniroyal Elec); Power Rating (none) -> 62.5 mW; Tolerance (none) -> ±1%; Voltage Rating (none) -> 50 V
- R17, R18, R2, R4, R6, R9: LCSC (none) -> C11702; MPN (none) -> 0402WGF1001TCE; Manufacturer (none) -> UNI-ROYAL(Uniroyal Elec); Power Rating (none) -> 62.5 mW; Tolerance (none) -> ±1%; Voltage Rating (none) -> 50 V
- R5: LCSC (none) -> C25105; MPN (none) -> 0402WGF330JTCE; Manufacturer (none) -> UNI-ROYAL(Uniroyal Elec); Power Rating (none) -> 62.5 mW; Tolerance (none) -> ±1%; Voltage Rating (none) -> 50 V
- SW1, SW2, SW3: LCSC (none) -> C92589; MPN (none) -> K2-1808SN-A4SW-01; Manufacturer (none) -> Korean Hroparts Elec
- U1: LCSC (none) -> C42411118; MPN (none) -> RP2350A; Manufacturer (none) -> Raspberry Pi
- U2: LCSC (none) -> C97521; MPN (none) -> W25Q128JVSIQ; Manufacturer (none) -> Winbond Elec
- U3: LCSC (none) -> C116706; MPN (none) -> MCP6002-I/SN; Manufacturer (none) -> Microchip Tech
- U4: LCSC (none) -> C92004; MPN (none) -> PT8211-S; Manufacturer (none) -> PTC(Princeton Tech)
- U6: Manufacturer Diodes -> Diodes Incorporated
- Y1: LCSC (none) -> C20625731; MPN (none) -> ABM8-272-T3; Manufacturer (none) -> Abracon LLC

Commit message: Add 16bit 5v as 2.0.0
Parts:
- D1: value LED -> KT-0603R; LCSC (none) -> C2286; MPN (none) -> KT-0603R; Manufacturer (none) -> Hubei KENTO Elec
- R7, R8: LCSC (none) -> C25100; MPN (none) -> 0402WGF270JTCE; Manufacturer (none) -> UNI-ROYAL(Uniroyal Elec); Power Rating (none) -> 62.5 mW; Tolerance (none) -> ±1%; Voltage Rating (none) -> 50 V
- U4: value PT8211-S -> TM8211-TA2302; LCSC C92004 -> C22381766; MPN PT8211-S -> TM8211-TA2302; Manufacturer PTC(Princeton Tech) -> TM(Shenzhen Titan Micro Elec)
- U5: value PSRAM -> APS6404L-3SQR-SN; LCSC (none) -> C5333729; MPN (none) -> APS6404L-3SQR-SN; Manufacturer (none) -> AP Memory
Other:
- note added: "## DAC 16-bit TM8211-TA2302 (PT8211-compatible) DAC."
- note added: "## PSRAM We are using Adafruit 4677 (64Mbit QSPI PSRAM, ESP-PSRAM64H class). Adafruit 4677 / LCSC C17430771 is out of stock, so this build is assembled with AP Memory APS6404L-3SQR-SN (LCSC C5333729), pin-identical SOP-8 QSPI PSRAM."
- note removed: "## DAC 16-bit PT8211 DAC."
- note removed: "## PSRAM We are using Adafruit 4677"
- moved on the sheet: C25, C26, C27, GND1, U6, V_SUPPLY1
